File: electronics/emc01/FPC EMC01 1284.brd (EAGLE design)
At the start: 160 x 100 mm, 111 parts, among them J4 PCIE, Q1 RFP30N06LE, Q2 RFP30N06LE, Q3 RFP30N06LE, SW1 SPST_TACT-EVQQ2, U1 LM2841, U10 MCP4728, U2 A4982, U3 A4982, U4 A4982, U5 ATMEGA1284P-AU, U6 A4982, U7 AP7313

Commit message: updated pinouts
Connections:
- removed net A-DIR: U6.14
- removed net A-STEP: U6.11
- removed net X-DIR: U2.14
- removed net X-STEP: U2.11
- removed net Y-DIR: U3.14
- removed net Y-STEP: U3.11
- removed net Z-DIR: U4.14
- removed net Z-STEP: U4.11
- new net A-ENABLE: U5.26
- new net A-STOP: U5.43
- new net DIR: U2.14, U3.14, U4.14, U5.22, U6.14
- new net PD0-RX1: U5.9
- new net PD1-TX1: U5.10
- new net PD2-RX2: U5.11
- new net PD3-TX2: U5.12
- new net STEP: U2.11, U3.11, U4.11, U5.21, U6.11
- new net X-ENABLE: U5.23
- new net Y-ENABLE: U5.24
- new net Z_ENABLE: U5.25
- net !HOTBED: now also U5.13
- net !HOTEND: now also U5.15
- net !PWM-FAN: now also U5.14
- net B-THERM: now also U5.37
- net E-THERM: now also U5.36
- net X-STOP: now also U5.40
- net Y-STOP: now also U5.41
- net Z-STOP: now also U5.42
Changed lines of the file:
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@@
 <contactref element="R9" pad="1"/>
 <contactref element="C10" pad="2"/>
-<wire x1="-42.28" y1="81.28" x2="-27.67" y2="93.98" width="0" layer="19" extent="1-1"/>
-<wire x1="-31.75" y1="60.96" x2="-42.28" y2="81.28" width="0" layer="19" extent="1-1"/>
+<contactref element="U5" pad="36"/>
+<wire x1="-31.75" y1="60.96" x2="76.369209375" y2="28.6073625" width="0" layer="19" extent="1-1"/>
+<wire x1="-42.28" y1="81.28" x2="-31.75" y2="60.96" width="0" layer="19" extent="1-1"/>
+<wire x1="-27.67" y1="93.98" x2="-42.28" y2="81.28" width="0" layer="19" extent="1-1"/>
 </signal>
 <signal name="B-THERM">
@@
 <contactref element="JP15" pad="1"/>
 <contactref element="C9" pad="2"/>
-<wire x1="-35.93" y1="81.28" x2="-32.75" y2="93.98" width="0" layer="19" extent="1-1"/>
-<wire x1="-21.59" y1="60.96" x2="-35.93" y2="81.28" width="0" layer="19" extent="1-1"/>
-</signal>
-<signal name="Y-STEP">
-<contactref element="U3" pad="11"/>
-</signal>
-<signal name="Y-DIR">
-<contactref element="U3" pad="14"/>
+<contactref element="U5" pad="37"/>
+<wire x1="-21.59" y1="60.96" x2="75.812434375" y2="28.0505875" width="0" layer="19" extent="1-1"/>
+<wire x1="-35.93" y1="81.28" x2="-21.59" y2="60.96" width="0" layer="19" extent="1-1"/>
+<wire x1="-32.75" y1="93.98" x2="-35.93" y2="81.28" width="0" layer="19" extent="1-1"/>
 </signal>
 <signal name="!HOTBED">
 <contactref element="R35" pad="1"/>
 <contactref element="R11" pad="1"/>
+<contactref element="U5" pad="13"/>
+<wire x1="-53.07" y1="93.98" x2="80.53605" y2="16.537896875" width="0" layer="19" extent="1-1"/>
 <wire x1="-61.96" y1="87.63" x2="-53.07" y2="93.98" width="0" layer="19" extent="1-1"/>
 </signal>
@@
 <contactref element="R6" pad="1"/>
 <contactref element="R36" pad="1"/>
+<contactref element="U5" pad="15"/>
+<wire x1="-73.39" y1="93.98" x2="81.6675625" y2="17.669409375" width="0" layer="19" extent="1-1"/>
 <wire x1="-94.98" y1="81.28" x2="-73.39" y2="93.98" width="0" layer="19" extent="1-1"/>
 </signal>
 <signal name="X-STOP">
 <contactref element="JP12" pad="P1"/>
+<contactref element="U5" pad="40"/>
+<wire x1="-56.3925" y1="30.5275" x2="74.124146875" y2="26.362296875" width="0" layer="19" extent="1-1"/>
 </signal>
 <signal name="Y-STOP">
 <contactref element="JP8" pad="P1"/>
+<contactref element="U5" pad="41"/>
+<wire x1="-38.6125" y1="30.5275" x2="73.549409375" y2="25.7875625" width="0" layer="19" extent="1-1"/>
 </signal>
 <signal name="Z-STOP">
 <contactref element="JP10" pad="P1"/>
-</signal>
-<signal name="X-STEP">
-<contactref element="U2" pad="11"/>
-</signal>
-<signal name="X-DIR">
-<contactref element="U2" pad="14"/>
-</signal>
-<signal name="Z-STEP">
-<contactref element="U4" pad="11"/>
-</signal>
-<signal name="Z-DIR">
-<contactref element="U4" pad="14"/>
+<contactref element="U5" pad="42"/>
+<wire x1="-47.5025" y1="30.5275" x2="72.992634375" y2="25.2307875" width="0" layer="19" extent="1-1"/>
 </signal>
 <signal name="SCLK">
@@
 <contactref element="R14" pad="1"/>
 <contactref element="Q3" pad="1"/>
+<contactref element="U5" pad="14"/>
+<wire x1="-17.51" y1="87.63" x2="81.1107875" y2="17.112634375" width="0" layer="19" extent="1-1"/>
 <wire x1="-53.22" y1="61.91" x2="-17.51" y2="87.63" width="0" layer="19" extent="1-1"/>
 </signal>
@@
 <wire x1="-137.51" y1="-128.83" x2="-135.001" y2="-151.13" width="0" layer="19" extent="1-1"/>
 </signal>
-<signal name="A-DIR">
-<contactref element="U6" pad="14"/>
-</signal>
-<signal name="A-STEP">
-<contactref element="U6" pad="11"/>
-</signal>
 <signal name="!A-ENABLE">
 <contactref element="U6" pad="23"/>
@@
 <wire x1="-42.26" y1="55.07" x2="-70.87" y2="30.5275" width="0" layer="19" extent="1-1"/>
 </signal>
+<signal name="N$26">
+<contactref element="U3" pad="15"/>
+<contactref element="JP1" pad="P2"/>
+<wire x1="-39.66" y1="55.07" x2="-68.87" y2="30.5275" width="0" layer="19" extent="1-1"/>
+</signal>
+<signal name="N$31">
+<contactref element="U3" pad="22"/>
+<contactref element="JP1" pad="P1"/>
+<wire x1="-44.21" y1="55.07" x2="-66.87" y2="30.5275" width="0" layer="19" extent="1-1"/>
+</signal>
+<signal name="N$39">
+<contactref element="U4" pad="18"/>
+<contactref element="JP3" pad="P4"/>
+<wire x1="-54.31" y1="55.07" x2="-84.3" y2="30.5275" width="0" layer="19" extent="1-1"/>
+</signal>
+<signal name="N$40">
+<contactref element="U4" pad="19"/>
+<contactref element="JP3" pad="P3"/>
+<wire x1="-54.96" y1="55.07" x2="-82.3" y2="30.5275" width="0" layer="19" extent="1-1"/>
+</signal>
+<signal name="N$41">
+<contactref element="U4" pad="15"/>
+<contactref element="JP3" pad="P2"/>
+<wire x1="-52.36" y1="55.07" x2="-80.3" y2="30.5275" width="0" layer="19" extent="1-1"/>
+</signal>
+<signal name="N$53">
+<contactref element="U4" pad="22"/>
+<contactref element="JP3" pad="P1"/>
+<wire x1="-56.91" y1="55.07" x2="-78.3" y2="30.5275" width="0" layer="19" extent="1-1"/>
+</signal>
+<signal name="N$56">
+<contactref element="U6" pad="18"/>
+<contactref element="JP11" pad="P4"/>
+<wire x1="-136.86" y1="-122.73" x2="-141.45" y2="-134.5725" width="0" layer="19" extent="1-1"/>
+</signal>
+<signal name="N$59">
+<contactref element="U6" pad="19"/>
+<contactref element="JP11" pad="P3"/>
+<wire x1="-137.51" y1="-122.73" x2="-139.45" y2="-134.5725" width="0" layer="19" extent="1-1"/>
+</signal>
+<signal name="N$60">
+<contactref element="U6" pad="15"/>
+<contactref element="JP11" pad="P2"/>
+<wire x1="-134.91" y1="-122.73" x2="-137.45" y2="-134.5725" width="0" layer="19" extent="1-1"/>
+</signal>
+<signal name="N$61">
+<contactref element="U6" pad="22"/>
+<contactref element="JP11" pad="P1"/>
+<wire x1="-139.46" y1="-122.73" x2="-135.45" y2="-134.5725" width="0" layer="19" extent="1-1"/>
+</signal>
+<signal name="Z_ENABLE">
+<contactref element="U5" pad="25"/>
+</signal>
+<signal name="A-ENABLE">
+<contactref element="U5" pad="26"/>
+</signal>
+<signal name="Y-ENABLE">
+<contactref element="U5" pad="24"/>
+</signal>
+<signal name="X-ENABLE">
+<contactref element="U5" pad="23"/>
+</signal>
+<signal name="DIR">
+<contactref element="U5" pad="22"/>
+<contactref element="U4" pad="14"/>
+<contactref element="U6" pad="14"/>
+<contactref element="U3" pad="14"/>
+<contactref element="U2" pad="14"/>
+<wire x1="-26.31" y1="55.07" x2="85.618875" y2="21.620721875" width="0" layer="19" extent="1-1"/>
+<wire x1="-39.01" y1="55.07" x2="-26.31" y2="55.07" width="0" layer="19" extent="1-1"/>
+<wire x1="-51.71" y1="55.07" x2="-39.01" y2="55.07" width="0" layer="19" extent="1-1"/>
+<wire x1="-134.26" y1="-122.73" x2="-51.71" y2="55.07" width="0" layer="19" extent="1-1"/>
+</signal>
+<signal name="STEP">
+<contactref element="U5" pad="21"/>
+<contactref element="U4" pad="11"/>
+<contactref element="U6" pad="11"/>
+<contactref element="U3" pad="11"/>
+<contactref element="U2" pad="11"/>
+<wire x1="-26.31" y1="48.97" x2="85.0621" y2="21.063946875" width="0" layer="19" extent="1-1"/>
+<wire x1="-39.01" y1="48.97" x2="-26.31" y2="48.97" width="0" layer="19" extent="1-1"/>
+<wire x1="-51.71" y1="48.97" x2="-39.01" y2="48.97" width="0" layer="19" extent="1-1"/>
+<wire x1="-134.26" y1="-128.83" x2="-51.71" y2="48.97" width="0" layer="19" extent="1-1"/>
+</signal>
 <signal name="N$25">
 <contactref element="U3" pad="18"/>
@@
 <wire x1="-41.61" y1="55.07" x2="-72.87" y2="30.5275" width="0" layer="19" extent="1-1"/>
 </signal>
-<signal name="N$26">
-<contactref element="U3" pad="15"/>
-<contactref element="JP1" pad="P2"/>
-<wire x1="-39.66" y1="55.07" x2="-68.87" y2="30.5275" width="0" layer="19" extent="1-1"/>
-</signal>
-<signal name="N$31">
-<contactref element="U3" pad="22"/>
-<contactref element="JP1" pad="P1"/>
-<wire x1="-44.21" y1="55.07" x2="-66.87" y2="30.5275" width="0" layer="19" extent="1-1"/>
-</signal>
-<signal name="N$39">
-<contactref element="U4" pad="18"/>
-<contactref element="JP3" pad="P4"/>
-<wire x1="-54.31" y1="55.07" x2="-84.3" y2="30.5275" width="0" layer="19" extent="1-1"/>
-</signal>
-<signal name="N$40">
-<contactref element="U4" pad="19"/>
-<contactref element="JP3" pad="P3"/>
-<wire x1="-54.96" y1="55.07" x2="-82.3" y2="30.5275" width="0" layer="19" extent="1-1"/>
-</signal>
-<signal name="N$41">
-<contactref element="U4" pad="15"/>
-<contactref element="JP3" pad="P2"/>
-<wire x1="-52.36" y1="55.07" x2="-80.3" y2="30.5275" width="0" layer="19" extent="1-1"/>
-</signal>
-<signal name="N$53">
-<contactref element="U4" pad="22"/>
-<contactref element="JP3" pad="P1"/>
-<wire x1="-56.91" y1="55.07" x2="-78.3" y2="30.5275" width="0" layer="19" extent="1-1"/>
-</signal>
-<signal name="N$56">
-<contactref element="U6" pad="18"/>
-<contactref element="JP11" pad="P4"/>
-<wire x1="-136.86" y1="-122.73" x2="-141.45" y2="-134.5725" width="0" layer="19" extent="1-1"/>
-</signal>
-<signal name="N$59">
-<contactref element="U6" pad="19"/>
-<contactref element="JP11" pad="P3"/>
-<wire x1="-137.51" y1="-122.73" x2="-139.45" y2="-134.5725" width="0" layer="19" extent="1-1"/>
-</signal>
-<signal name="N$60">
-<contactref element="U6" pad="15"/>
-<contactref element="JP11" pad="P2"/>
-<wire x1="-134.91" y1="-122.73" x2="-137.45" y2="-134.5725" width="0" layer="19" extent="1-1"/>
-</signal>
-<signal name="N$61">
-<contactref element="U6" pad="22"/>
-<contactref element="JP11" pad="P1"/>
-<wire x1="-139.46" y1="-122.73" x2="-135.45" y2="-134.5725" width="0" layer="19" extent="1-1"/>
+<signal name="A-STOP">
+<contactref element="U5" pad="43"/>
+</signal>
+<signal name="PD0-RX1">
+<contactref element="U5" pad="9"/>
+</signal>
+<signal name="PD1-TX1">
+<contactref element="U5" pad="10"/>
+</signal>
+<signal name="PD2-RX2">
+<contactref element="U5" pad="11"/>
+</signal>
+<signal name="PD3-TX2">
+<contactref element="U5" pad="12"/>
 </signal>
 </signals>

Commit message: updated pinouts
Parts:
- removed C10, C29, C9: 10uF, ipc-7351-capacitor:CAPC2012X145AN
- removed C23, C30, C37, C41: 0.1uF, ipc-7351-capacitor:CAPC2012X145AN
- removed C27: 0.22uF, ipc-7351-capacitor:CAPC2012X145AN
- removed C31: 100uF, rcl:PANASONIC_D
- removed JP11: MOT-Z, SRG:JST_B4B-PH_HEADER
- removed JP15: B-THERM, SparkFun:1X02
- removed JP16: E-THERM, SparkFun:1X02
- removed MS-Z1: (no value), printrbot:SJ_3_CONNECTED
- removed R10, R9: 4.7k, adafruit:R0805
- removed R13, R15: 0.11, adafruit:R0805
- removed R23: 10k, adafruit:R0805
- removed R29, R30: 100k, adafruit:R0805
- removed U6: A4982, printrbot:TSSOP-24
- added JP2: LCD HEADER, pinhead-2:2X08SMD
- added JP5: RPI GPIO, pinhead-2:2X13SMD
- added X1: Camera FFC, con-hirose:FH12-15S-0.5SH
- JP4: device printrbot:JP3Q -> pinhead-2:2X03SMD
Connections:
- net PD2-RX2 renamed TOOL4-ENABLE
- net PD3-TX2 renamed TOOL3-ENABLE
- removed net !A-ENABLE: R29.2, U6.23
- removed net !X-ENABLE: R3.2, U2.23
- removed net !Y-ENABLE: R21.2, U3.23
- removed net !Z-ENABLE: R27.2, U4.23
- removed net A-ENABLE: U5.26
- removed net A-STOP: U5.43
- removed net DIR: U2.14, U3.14, U4.14, U5.22, U6.14
- removed net N$1: LED1.A, R1.1
- removed net N$18: C27.2, U6.4
- removed net N$3: C23.2, U6.1
- removed net N$33: R30.2, U6.7, U6.9
- removed net N$4: C23.1, U6.2
- removed net N$48: C30.2, U6.3
- removed net N$54: MS-Z1.1, U6.5
- removed net N$55: MS-Z1.3, U6.6
- removed net N$56: JP11.P4, U6.18
- removed net N$59: JP11.P3, U6.19
- removed net N$6: R13.1, U6.17
- removed net N$60: JP11.P2, U6.15
- removed net N$61: JP11.P1, U6.22
- removed net N$8: R15.1, U6.20
- removed net N$9: R23.1, U6.8
- removed net STEP: U2.11, U3.11, U4.11, U5.21, U6.11
- removed net X-ENABLE: U5.23
- removed net Y-ENABLE: U5.24
- removed net Z_ENABLE: U5.25
- new net !XYZ-ENABLE: R21.2, R27.2, R3.2, U2.23, U3.23, U4.23
- new net TOOL-DIR: U5.40
- new net TOOL-STEP: U5.41
- new net TOOL1-DOUT: U5.33
- new net TOOL1-ENABLE: U5.14
- new net TOOL2-DOUT: U5.32
- new net TOOL2-ENABLE: U5.13
- new net TOOL3-DOUT: U5.31
- new net TOOL4-AIN: U5.34
- new net TOOL4-DOUT: U5.30
- new net X-DIR: U2.14, U5.24
- new net X-STEP: U2.11, U5.16
- new net XYZENABLE: U5.15
- new net Y-DIR: U3.14, U5.26
- new net Y-STEP: U3.11, U5.25
- new net Z-DIR: U4.14, U5.42
- new net Z-ENABLE: U5.35
- new net Z-STEP: U4.11, U5.43
- net !HOTBED: no longer U5.13
- net !HOTEND: no longer U5.15
- net !PWM-FAN: no longer U5.14
- net +5V: no longer C29.2, MS-Z1.2, R10.2, R29.1, R30.1, R9.2, U6.10
- net 12V: no longer C30.1, C31.+, C37.1, U6.16, U6.21
- net B-THERM: now also U5.36; no longer C9.2, JP15.1, R10.1, U5.37
- net E-THERM: now also U5.37; no longer C10.2, JP16.1, R9.1, U5.36
- net GND: no longer C10.1, C27.1, C29.1, C31.-, C37.2, C41.2, C9.1, JP15.2, JP16.2, R13.2, R15.2, R23.2, U6.13, U6.24, U6.PAD
- net VREF_Z: no longer C41.1, U6.12
- net X-STOP: now also U5.21; no longer U5.40
- net Y-STOP: now also U5.22; no longer U5.41
- net Z-STOP: now also U5.23; no longer U5.42

Commit message: updated pinouts
Parts:
- removed J2: (no value), printrbot:PHOENIX-5MM-2POS
- added CN1: (no value), adafruit:JST-PH-2-SMT-RA
- JP10, JP12, JP8: device SRG:JST_B3B-PH_HEADER -> adafruit:JSTPH3
- JP17: device SparkFun:1X02 -> adafruit:JST-PH-2-SMT
Connections:
- net +5V: now also JP10.2, JP12.2, JP8.2; no longer JP10.P2, JP12.P2, JP8.P2
- net 12V: now also CN1.2, JP17.2; no longer J2.P$1, JP17.1
- net GND: now also JP10.3, JP12.3, JP8.3; no longer JP10.P3, JP12.P3, JP8.P3
- net HOTBED-GND: now also CN1.1; no longer J2.P$2
- net N$5: now also JP17.1; no longer JP17.2
- net X-STOP: now also JP12.1; no longer JP12.P1
- net Y-STOP: now also JP8.1; no longer JP8.P1
- net Z-STOP: now also JP10.1; no longer JP10.P1
