File: electronics/emc01/FPC-EMC01-1284.brd (EAGLE design)
At the start: 100 x 86.6 mm, 52 parts, among them IC1 FT232RL, J10 ICSP, J11 CONN-RECT-16PIN-2ROW, J12 CONN-RECT-16PIN-2ROW, J13 CONN-RECT-16PIN-2ROW, J14 CONN-RECT-16PIN-2ROW, J2 PCIE, J4 MOT-X, J5 MOT-Y, J6 MOT-Z, J7 CONN-RECT-3PINJST_PH_2MM, J8 CONN-RECT-3PINJST_PH_2MM, J9 CONN-RECT-3PINJST_PH_2MM, Q4 16Mhz, U1 STEPSTICK, U2 STEPSTICK, U3 STEPSTICK, U5 ATMEGA1284P-AU, U6 LM2576-D2T, X1 USB-MICROB

Commit message: emc01 routing update
Routing:
- net N$9: track 0.00 -> 20.8 mm
- net N$7: track 0.00 -> 20.2 mm
- net N$8: track 0.00 -> 20.2 mm, vias 0 -> 1
- net N$6: track 0.00 -> 19.5 mm, vias 0 -> 1
- net N$15: track 11.1 -> 12.7 mm
Changed lines of the file:
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@@
 <wire x1="11.5697375" y1="59.879146875" x2="9.12" y2="57.429409375" width="0.4064" layer="1"/>
 <wire x1="9.12" y1="57.429409375" x2="9.12" y2="49.514" width="0.4064" layer="1"/>
+<wire x1="82.9" y1="49.032" x2="79.485259375" y2="45.617259375" width="1.016" layer="1"/>
+<wire x1="79.485259375" y1="45.617259375" x2="79.485259375" y2="43.387965625" width="1.016" layer="1"/>
 <wire x1="66.7717375" y1="71.99285" x2="75.806" y2="84.836" width="0" layer="19" extent="1-1"/>
 <wire x1="68.0417375" y1="69.793146875" x2="66.7717375" y2="71.99285" width="0" layer="19" extent="1-1"/>
@@
 <wire x1="29.3047375" y1="27.99003125" x2="9.12" y2="49.514" width="0" layer="19" extent="1-1"/>
 <wire x1="46.596" y1="16.67" x2="29.3047375" y2="27.99003125" width="0" layer="19" extent="1-1"/>
-<wire x1="82.9" y1="49.032" x2="79.485259375" y2="45.617259375" width="1.016" layer="1"/>
-<wire x1="79.485259375" y1="45.617259375" x2="79.485259375" y2="43.387965625" width="1.016" layer="1"/>
 </signal>
 <signal name="MISO">
@@
 <contactref element="U1" pad="2B"/>
 <contactref element="J4" pad="4"/>
-<wire x1="33" y1="85.57" x2="46.49" y2="76.921" width="0" layer="19" extent="1-1"/>
+<wire x1="33" y1="85.57" x2="33" y2="83.1" width="1.016" layer="1"/>
+<via x="33" y="83.1" extent="1-16" drill="0.6" shape="octagon"/>
+<wire x1="33" y1="83.1" x2="35.9" y2="80.2" width="1.016" layer="16"/>
+<wire x1="35.9" y1="80.2" x2="44.85" y2="80.2" width="1.016" layer="16"/>
+<wire x1="44.85" y1="80.2" x2="46.49" y2="78.56" width="1.016" layer="16"/>
+<wire x1="46.49" y1="78.56" x2="46.49" y2="76.921" width="1.016" layer="16"/>
 </signal>
 <signal name="N$7">
 <contactref element="J4" pad="3"/>
 <contactref element="U1" pad="2A"/>
-<wire x1="35" y1="85.57" x2="49.03" y2="76.921" width="0" layer="19" extent="1-1"/>
+<wire x1="35" y1="85.57" x2="35" y2="82.75" width="1.016" layer="1"/>
+<wire x1="35" y1="82.75" x2="36.15" y2="81.45" width="1.016" layer="1"/>
+<wire x1="36.15" y1="81.45" x2="38.3" y2="81.45" width="1.016" layer="1"/>
+<wire x1="38.3" y1="81.45" x2="38.95" y2="81.9" width="1.016" layer="1"/>
+<wire x1="38.95" y1="81.9" x2="40.65" y2="81.9" width="1.016" layer="1"/>
+<wire x1="40.65" y1="81.9" x2="42.5" y2="80.2" width="1.016" layer="1"/>
+<wire x1="42.5" y1="80.2" x2="46.85" y2="80.2" width="1.016" layer="1"/>
+<wire x1="46.85" y1="80.2" x2="49.03" y2="78.02" width="1.016" layer="1"/>
+<wire x1="49.03" y1="78.02" x2="49.03" y2="76.921" width="1.016" layer="1"/>
 </signal>
 <signal name="N$8">
 <contactref element="U1" pad="1A"/>
 <contactref element="J4" pad="2"/>
-<wire x1="37" y1="85.57" x2="51.57" y2="76.921" width="0" layer="19" extent="1-1"/>
+<wire x1="37" y1="85.57" x2="36.95" y2="85.52" width="1.016" layer="1"/>
+<wire x1="36.95" y1="85.52" x2="36.95" y2="82.85" width="1.016" layer="1"/>
+<via x="36.95" y="82.85" extent="1-16" drill="0.6" shape="octagon"/>
+<wire x1="36.95" y1="82.85" x2="37.9" y2="81.9" width="1.016" layer="16"/>
+<wire x1="37.9" y1="81.9" x2="47.2" y2="81.9" width="1.016" layer="16"/>
+<wire x1="47.2" y1="81.9" x2="51.57" y2="77.53" width="1.016" layer="16"/>
+<wire x1="51.57" y1="77.53" x2="51.57" y2="76.921" width="1.016" layer="16"/>
 </signal>
 <signal name="N$9">
 <contactref element="J4" pad="1"/>
 <contactref element="U1" pad="1B"/>
-<wire x1="39" y1="85.57" x2="54.11" y2="76.921" width="0" layer="19" extent="1-1"/>
+<wire x1="43.22" y1="81.75" x2="50.9" y2="81.9" width="1.016" layer="1"/>
+<wire x1="50.9" y1="81.9" x2="54.11" y2="78.69" width="1.016" layer="1"/>
+<wire x1="54.11" y1="78.69" x2="54.11" y2="76.921" width="1.016" layer="1"/>
+<wire x1="43.22" y1="81.75" x2="41.22" y2="83.75" width="1.016" layer="1"/>
+<wire x1="41.22" y1="83.75" x2="39.1" y2="83.75" width="1.016" layer="1"/>
+<wire x1="39.1" y1="83.75" x2="39" y2="83.85" width="1.016" layer="1"/>
+<wire x1="39" y1="83.85" x2="39" y2="85.57" width="1.016" layer="1"/>
 </signal>
 <signal name="N$11">
@@
 <contactref element="U2" pad="2B"/>
 <contactref element="J5" pad="4"/>
-<wire x1="24.291440625" y1="23.385921875" x2="26.35" y2="24.65" width="1.016" layer="1"/>
-<via x="26.35" y="24.65" extent="1-16" drill="0.6" shape="octagon"/>
-<wire x1="26.35" y1="24.65" x2="26.3" y2="29" width="1.016" layer="16"/>
-<wire x1="26.3" y1="29" x2="24.95" y2="30.35" width="1.016" layer="16"/>
-<wire x1="24.95" y1="30.35" x2="25.55" y2="31.024703125" width="1.016" layer="16"/>
-<wire x1="25.55" y1="31.024703125" x2="26.7647375" y2="32.389440625" width="1.016" layer="16"/>
+<wire x1="24.291440625" y1="23.385921875" x2="26.45" y2="24.65" width="1.016" layer="1"/>
+<via x="26.45" y="24.65" extent="1-16" drill="0.6" shape="octagon"/>
+<wire x1="26.45" y1="24.65" x2="26.6" y2="27.7" width="1.016" layer="16"/>
+<wire x1="26.6" y1="27.7" x2="26.3" y2="28.25" width="1.016" layer="16"/>
+<wire x1="26.3" y1="28.25" x2="25" y2="30.2" width="1.016" layer="16"/>
+<wire x1="25" y1="30.2" x2="25.35" y2="31.474703125" width="1.016" layer="16"/>
+<wire x1="25.35" y1="31.474703125" x2="26.7647375" y2="32.389440625" width="1.016" layer="16"/>
 </signal>
 <signal name="N$13">
 <contactref element="U2" pad="2A"/>
 <contactref element="J5" pad="3"/>
-<wire x1="23.291440625" y1="25.117971875" x2="26.3" y2="27.05" width="1.016" layer="1"/>
-<wire x1="26.3" y1="27.05" x2="26.3" y2="29" width="1.016" layer="1"/>
-<wire x1="26.3" y1="29" x2="24.15" y2="31.15" width="1.016" layer="1"/>
-<wire x1="24.15" y1="31.15" x2="24.15" y2="33.244409375" width="1.016" layer="1"/>
-<wire x1="24.15" y1="33.244409375" x2="25.4947375" y2="34.589146875" width="1.016" layer="1"/>
+<wire x1="23.291440625" y1="25.117971875" x2="25.85" y2="26.65" width="1.016" layer="1"/>
+<wire x1="25.85" y1="26.65" x2="26.25" y2="28.05" width="1.016" layer="1"/>
+<wire x1="26.25" y1="28.05" x2="23.65" y2="32" width="1.016" layer="1"/>
+<wire x1="23.65" y1="32" x2="24.1" y2="33.794409375" width="1.016" layer="1"/>
+<wire x1="24.1" y1="33.794409375" x2="25.4947375" y2="34.589146875" width="1.016" layer="1"/>
 </signal>
 <signal name="N$14">
 <contactref element="U2" pad="1A"/>
 <contactref element="J5" pad="2"/>
-<wire x1="22.291440625" y1="26.850025" x2="24.55" y2="28.2" width="1.016" layer="1"/>
-<via x="24.55" y="28.2" extent="1-16" drill="0.6" shape="octagon"/>
-<wire x1="24.55" y1="28.2" x2="22.4" y2="30.35" width="1.016" layer="16"/>
-<wire x1="22.4" y1="30.35" x2="22.4" y2="34.7" width="1.016" layer="16"/>
-<wire x1="22.4" y1="34.7" x2="24.2247375" y2="36.5247375" width="1.016" layer="16"/>
-<wire x1="24.2247375" y1="36.5247375" x2="24.2247375" y2="36.78885" width="1.016" layer="16"/>
+<wire x1="22.291440625" y1="26.850025" x2="24.3" y2="28.1" width="1.016" layer="1"/>
+<via x="24.3" y="28.1" extent="1-16" drill="0.6" shape="octagon"/>
+<wire x1="24.3" y1="28.1" x2="21.8" y2="31.55" width="1.016" layer="16"/>
+<wire x1="21.8" y1="31.55" x2="21.5" y2="34.4" width="1.016" layer="16"/>
+<wire x1="21.5" y1="34.4" x2="22.63885" y2="36.18885" width="1.016" layer="16"/>
+<wire x1="22.63885" y1="36.18885" x2="24.2247375" y2="36.78885" width="1.016" layer="16"/>
 </signal>
 <signal name="N$15">
 <contactref element="U2" pad="1B"/>
 <contactref element="J5" pad="1"/>
-<wire x1="21.291440625" y1="28.582075" x2="21.291440625" y2="37.325259375" width="1.016" layer="1"/>
-<wire x1="21.291440625" y1="37.325259375" x2="22.9547375" y2="38.98855625" width="1.016" layer="1"/>
+<wire x1="22.9547375" y1="38.98855625" x2="21.1" y2="37.93381875" width="1.016" layer="1"/>
+<wire x1="21.1" y1="37.93381875" x2="21.5" y2="31.45" width="1.016" layer="1"/>
+<wire x1="21.5" y1="31.45" x2="22.8" y2="29.55" width="1.016" layer="1"/>
+<wire x1="22.8" y1="29.55" x2="21.291440625" y2="28.582075" width="1.016" layer="1"/>
 </signal>
 <signal name="N$16">

Commit message: polygonception
Parts:
- moved R5 37.9 mm to (43.4, 43.6), turned to 180 degrees
- moved J3 32.9 mm to (34.1, 59.5), turned to 60 degrees
- moved R4 5.93 mm to (63.2, 48.0)
- moved C2 2.22 mm to (23.8, 13.3), turned to 90 degrees
- moved C10 1.03 mm to (44.1, 18.1)
Routing:
- net 12V: track 18.4 -> 117.8 mm, vias 0 -> 1
- net SDA: track 0.00 -> 66.6 mm, vias 0 -> 2
- net SCL: track 0.00 -> 65.8 mm, vias 0 -> 2
- net Y-STOP: track 0.00 -> 46.5 mm, vias 0 -> 2
- net !RESET: track 0.00 -> 33.5 mm
- net !XYZ-ENABLE: track 20.9 -> 16.2 mm
- net DTR: track 0.00 -> 4.00 mm
- net GND: track 17.7 -> 14.7 mm
- net N$15: track 12.7 -> 12.1 mm
- added copper zone on layer 1, net 12V

Commit message: routing update
Parts:
- moved C7 55.4 mm to (50.9, 34.3), turned to 180 degrees
- moved R5 33.7 mm to (31.7, 12.0), turned to 0 degrees
- moved R3 13.4 mm to (51.0, 38.8), turned to 0 degrees
- moved C3 8.26 mm to (45.1, 40.7)
- moved C2 7.08 mm to (30.7, 14.9)
- moved C11 6.67 mm to (40.7, 41.6), turned to 180 degrees
- moved Q4 6.32 mm to (44.1, 37.7)
- moved R4 5.85 mm to (66.8, 52.6), turned to 180 degrees
- moved C16 3.02 mm to (14.5, 48.9), turned to 300 degrees
- moved C18 1.14 mm to (85.6, 50.1), turned to 210 degrees
- moved R1 1.00 mm to (38.4, 57.9)
- moved D1 0.90 mm to (65.5, 20.2)
- moved C34 0.71 mm to (38.5, 49.8)
- moved U6 0.63 mm to (50.2, 26.4)
- moved C13 0.51 mm to (38.4, 55.2)
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Connections:
- net SCL: now also JP5.3; no longer JP5.4
- net SDA: now also JP5.4; no longer JP5.3
Routing:
- net AVR_TXD: track 0.00 -> 138.6 mm, vias 0 -> 3
- net AVR_RXD: track 0.00 -> 138.3 mm, vias 0 -> 3
- net 12V: track 117.8 -> 221.9 mm, vias 1 -> 20
- net SCL: track 65.8 -> 163.7 mm, vias 2 -> 3
- net TOOL_STEP: track 0.00 -> 93.8 mm, vias 0 -> 3
- net !RESET: track 33.5 -> 90.8 mm, vias 0 -> 3
- net TOOL3_DOUT: track 0.00 -> 57.3 mm
- net DTR: track 4.00 -> 59.5 mm
- net MOSI: track 0.00 -> 50.9 mm, vias 0 -> 2
- net X-STOP: track 0.00 -> 48.8 mm, vias 0 -> 2
- net MISO: track 0.00 -> 46.0 mm, vias 0 -> 1
- net Z-STOP: track 0.00 -> 42.2 mm
- net TOOL2_DOUT: track 0.00 -> 39.0 mm, vias 0 -> 1
- net SDA: track 66.6 -> 101.8 mm, vias 2 -> 4
- net Z_STEP: track 0.00 -> 30.3 mm, vias 0 -> 1
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- added copper zone on layer 16, net 12V
