File: electronics/emc01/FPC-EMC01-1284.sch (EAGLE design)
At the start: 75 parts, among them J1 USB-MINIB-5PIN, J10 CONN-OSTTA020161, J11 CONN-RECT-16PIN-2ROW, J12 CONN-RECT-16PIN-2ROW, J13 CONN-RECT-16PIN-2ROW, J14 CONN-RECT-16PIN-2ROW, J15 DNP, J16 ICSP, J3 DNP, J4A MOT-X, J5A MOT-Y, J6A MOT-Z, J7A CONN-RECT-3PINJST_PH_2MM, J8A CONN-RECT-3PINJST_PH_2MM, J9A CONN-RECT-3PINJST_PH_2MM, Q2 2N7002PW, U1 IC-ATMEGA1284P-AU, U2 FT231XS, X1 16Mhz

Commit message: minor cosmetic and refdes updates
Parts:
- renumbered IC1 to U3
Changed lines of the file:
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@@
 <part name="P+6" library="supply1" deviceset="+5V" device=""/>
 <part name="P+7" library="supply1" deviceset="+5V" device=""/>
-<part name="IC1" library="SparkFun-PowerIC" deviceset="V_REG_LM1117" device="SOT223"/>
+<part name="U3" library="SparkFun-PowerIC" deviceset="V_REG_LM1117" device="SOT223"/>
 <part name="GND13" library="supply1" deviceset="GND" device=""/>
 <part name="P+8" library="supply1" deviceset="+5V" device=""/>
@@
 <attribute name="VALUE" x="87.63" y="177.8" size="1.778" layer="96"/>
 </instance>
-<instance part="IC1" gate="G$1" x="214.63" y="218.44"/>
+<instance part="U3" gate="G$1" x="214.63" y="218.44"/>
 <instance part="GND13" gate="1" x="214.63" y="199.39"/>
 <instance part="P+8" gate="1" x="234.95" y="232.41" smashed="yes">
@@
 </segment>
 <segment>
-<pinref part="IC1" gate="G$1" pin="ADJ"/>
+<pinref part="U3" gate="G$1" pin="ADJ"/>
 <pinref part="GND13" gate="1" pin="GND"/>
 <wire x1="214.63" y1="210.82" x2="214.63" y2="201.93" width="0.1524" layer="91"/>
@@
 </segment>
 <segment>
-<pinref part="IC1" gate="G$1" pin="IN"/>
+<pinref part="U3" gate="G$1" pin="IN"/>
 <pinref part="U$15" gate="G$1" pin="12V"/>
 <wire x1="207.01" y1="218.44" x2="201.93" y2="218.44" width="0.1524" layer="91"/>
@@
 <segment>
 <pinref part="P+8" gate="1" pin="+5V"/>
-<pinref part="IC1" gate="G$1" pin="OUT@1"/>
+<pinref part="U3" gate="G$1" pin="OUT@1"/>
 <wire x1="234.95" y1="215.9" x2="234.95" y2="229.87" width="0.1524" layer="91"/>
 <wire x1="222.25" y1="215.9" x2="227.33" y2="215.9" width="0.1524" layer="91"/>
@@
 <wire x1="234.95" y1="212.09" x2="234.95" y2="215.9" width="0.1524" layer="91"/>
 <junction x="234.95" y="215.9"/>
-<pinref part="IC1" gate="G$1" pin="OUT"/>
+<pinref part="U3" gate="G$1" pin="OUT"/>
 <wire x1="222.25" y1="218.44" x2="227.33" y2="218.44" width="0.1524" layer="91"/>
 <wire x1="227.33" y1="218.44" x2="227.33" y2="215.9" width="0.1524" layer="91"/>

Commit message: Moving STL's over here
Parts:
- added U4: IC-ATMEGA1284P-AU, FirePick:IC-ATMEGA1284P-AU
Other:
- note added: "ARDUINO PIN MAPPING -----------------------------------------"
- note added: "Revision A: First official release. Revision B: Added voltage regulator. Moved vias. Updated silkscreen. Revision C: Fixed air-wire @ C3/C11 to GND (Thanks, Douglas!)"
- note added: "Revision C"
- note removed: "Revision B"
Changed lines of the file:
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@@
 <?xml version="1.0" encoding="utf-8"?>
 <!DOCTYPE eagle SYSTEM "eagle.dtd">
-<eagle version="7.1.0">
+<eagle version="7.2.0">
 <drawing>
 <settings>
@@
 <part name="GND14" library="supply1" deviceset="GND" device=""/>
 <part name="J10" library="FirePick" deviceset="CONN-OSTTA020161" device=""/>
+<part name="U4" library="FirePick" deviceset="IC-ATMEGA1284P-AU" device=""/>
 </parts>
 <sheets>
@@
 <text x="289.56" y="20.32" size="1.778" layer="94" ratio="15">Drawn by: NEIL JANSEN</text>
 <text x="289.56" y="16.51" size="1.778" layer="94" ratio="15">Checked  by:</text>
-<text x="290.83" y="7.62" size="2.54" layer="94" ratio="10">Revision B</text>
+<text x="290.83" y="7.62" size="2.54" layer="94" ratio="10">Revision C</text>
 <wire x1="5.715" y1="28.575" x2="288.29" y2="28.575" width="0.3048" layer="94"/>
 <wire x1="288.29" y1="28.575" x2="288.29" y2="3.81" width="0.3048" layer="94"/>
@@
 <text x="5.08" y="30.48" size="1.778" layer="95">Released under the Creative Commons Attribution Share-Alike 4.0 License</text>
 <text x="207.01" y="226.06" size="5.08" layer="94">VREG</text>
+<text x="299.72" y="40.64" size="1.778" layer="91">Revision A: First official release.
+Revision B: Added voltage regulator.
+    Moved vias.  Updated silkscreen.
+Revision C: Fixed air-wire @ C3/C11 to
+    GND (Thanks, Douglas!)</text>
 </plain>
 <instances>
@@
 </nets>
 </sheet>
+<sheet>
+<plain>
+<text x="10.16" y="68.58" size="1.778" layer="91">ARDUINO PIN MAPPING
+-----------------------------------------
+</text>
+</plain>
+<instances>
+<instance part="U4" gate="G$1" x="-35.56" y="67.31"/>
+</instances>
+<busses>
+</busses>
+<nets>
+</nets>
+</sheet>
