File: electronics/ehdmifpc01/FireExtender.sch (KiCad schematic (older format))
At the start: 4 parts, among them J1 MOLEX_47151-1101, J2 CONN_15_RPI-CAM

Commit message: Changed to correct pinout for Type A HDMI
Parts:
- removed J1: MOLEX_47151-1101, ~, symbol MOLEX_46765-1302
- added J1: HDMI_TYPE_A, ~, symbol HDMI_TYPE_A
Connections:
- net labels added: +3V3, CLK+, CLK-, D0+, D0-, D1+, D1-, D2+, D2-, SCL, SDA
- wire segments 40 -> 39
Changed lines of the file:
@@
 Sheet 1 1
 Title "HDMI to FPC for RPi Cam"
-Date "16 jun 2014"
+Date "27 aug 2014"
 Rev "A"
 Comp "Firepick"
@@
 Comment4 ""
 $EndDescr
-$Comp
-L MOLEX_46765-1302 J1
-U 1 1 539F1EB1
-P 4800 3350
-F 0 "J1" H 4800 4500 60  0000 C CNN
-F 1 "MOLEX_47151-1101" H 4800 4600 60  0000 C CNN
-F 2 "~" H 4450 4000 60  0000 C CNN
-F 3 "~" H 4450 4000 60  0000 C CNN
-	1    4800 3350
-	-1   0    0    -1
-$EndComp
 $Comp
 L C C1
@@
 L GND #PWR01
 U 1 1 539F1F4C
-P 5400 4400
-F 0 "#PWR01" H 5400 4400 30  0001 C CNN
-F 1 "GND" H 5400 4330 30  0001 C CNN
-F 2 "" H 5400 4400 60  0000 C CNN
-F 3 "" H 5400 4400 60  0000 C CNN
-	1    5400 4400
+P 5400 4750
+F 0 "#PWR01" H 5400 4750 30  0001 C CNN
+F 1 "GND" H 5400 4680 30  0001 C CNN
+F 2 "" H 5400 4750 60  0000 C CNN
+F 3 "" H 5400 4750 60  0000 C CNN
+	1    5400 4750
 	1    0    0    -1
 $EndComp
@@
 	1    0    0    -1
 $EndComp
-Wire Wire Line
-	5300 2700 5400 2700
-Wire Wire Line
-	5400 2700 5400 4400
-Wire Wire Line
-	5300 3000 5400 3000
-Connection ~ 5400 3000
-Wire Wire Line
-	5300 3300 5400 3300
-Connection ~ 5400 3300
-Wire Wire Line
-	5300 3600 5400 3600
-Connection ~ 5400 3600
-Wire Wire Line
-	5300 3900 5400 3900
-Connection ~ 5400 3900
-Wire Wire Line
-	7350 2600 7250 2600
-Wire Wire Line
-	7250 2600 7250 4100
-Wire Wire Line
-	7350 2900 7250 2900
-Connection ~ 7250 2900
-Wire Wire Line
-	7350 3200 7250 3200
-Connection ~ 7250 3200
-Wire Wire Line
-	7350 3500 7250 3500
-Connection ~ 7250 3500
-Wire Wire Line
-	5300 4200 6400 4200
-Wire Wire Line
-	6400 4200 6400 4000
-Wire Wire Line
-	6400 4000 7350 4000
-Wire Wire Line
-	7350 3900 6300 3900
-Wire Wire Line
-	6300 3900 6300 4100
-Wire Wire Line
-	6300 4100 5300 4100
-Wire Wire Line
-	5300 4000 6200 4000
-Wire Wire Line
-	6200 4000 6200 3800
-Wire Wire Line
-	6200 3800 7350 3800
-Wire Wire Line
-	7100 4300 7100 4000
-Connection ~ 7100 4000
-Wire Wire Line
-	5650 4300 5650 4200
-Connection ~ 5650 4200
 $Comp
 L GND #PWR03
@@
 	1    0    0    -1
 $EndComp
-Wire Wire Line
-	5650 4700 5650 4750
 $Comp
 L GND #PWR04
@@
 	1    0    0    -1
 $EndComp
-Wire Wire Line
-	7100 4700 7100 4750
-Wire Wire Line
-	5300 3700 7350 3700
-Wire Wire Line
-	6300 3600 7350 3600
-Wire Wire Line
-	7350 2700 6300 2700
-Wire Wire Line
-	6300 2700 6300 2600
-Wire Wire Line
-	6300 2600 5300 2600
-Wire Wire Line
-	5300 2800 7350 2800
-Wire Wire Line
-	7350 3000 6300 3000
-Wire Wire Line
-	6300 3000 6300 2900
-Wire Wire Line
-	6300 2900 5300 2900
-Wire Wire Line
-	5300 3100 7350 3100
-Wire Wire Line
-	7350 3300 6300 3300
-Wire Wire Line
-	6300 3300 6300 3200
-Wire Wire Line
-	6300 3200 5300 3200
-Wire Wire Line
-	5300 3400 7350 3400
-Wire Wire Line
-	6300 3600 6300 3500
-Wire Wire Line
-	6300 3500 5300 3500
 Text Notes 5900 2050 0    59   ~ 0
 HDMI to FPC connector \nfor RPi CAM
+$Comp
+L HDMI_TYPE_A J1
+U 1 1 53FE06C7
+P 4800 3550
+F 0 "J1" H 4800 4700 60  0000 C CNN
+F 1 "HDMI_TYPE_A" H 4800 4800 60  0000 C CNN
+F 2 "~" H 4450 4200 60  0000 C CNN
+F 3 "~" H 4450 4200 60  0000 C CNN
+	1    4800 3550
+	-1   0    0    -1
+$EndComp
+Wire Wire Line
+	5300 2700 5400 2700
+Wire Wire Line
+	5400 2700 5400 4750
+Wire Wire Line
+	5300 3000 5400 3000
+Connection ~ 5400 3000
+Wire Wire Line
+	5300 3300 5400 3300
+Connection ~ 5400 3300
+Wire Wire Line
+	5300 3600 5400 3600
+Connection ~ 5400 3600
+Wire Wire Line
+	7350 2600 7250 2600
+Wire Wire Line
+	7250 2600 7250 4100
+Wire Wire Line
+	7350 2900 7250 2900
+Connection ~ 7250 2900
+Wire Wire Line
+	7350 3200 7250 3200
+Connection ~ 7250 3200
+Wire Wire Line
+	7350 3500 7250 3500
+Connection ~ 7250 3500
+Wire Wire Line
+	6400 4000 7350 4000
+Wire Wire Line
+	7350 3900 6300 3900
+Wire Wire Line
+	6300 3900 6300 4100
+Wire Wire Line
+	6300 4100 5300 4100
+Wire Wire Line
+	5300 4000 6200 4000
+Wire Wire Line
+	6200 4000 6200 3800
+Wire Wire Line
+	6200 3800 7350 3800
+Wire Wire Line
+	7100 4300 7100 4000
+Connection ~ 7100 4000
+Wire Wire Line
+	5650 4700 5650 4750
+Wire Wire Line
+	7100 4700 7100 4750
+Wire Wire Line
+	5300 3700 7350 3700
+Wire Wire Line
+	6300 3600 7350 3600
+Wire Wire Line
+	7350 2700 6300 2700
+Wire Wire Line
+	6300 2700 6300 2600
+Wire Wire Line
+	6300 2600 5300 2600
+Wire Wire Line
+	5300 2800 7350 2800
+Wire Wire Line
+	7350 3000 6300 3000
+Wire Wire Line
+	6300 3000 6300 2900
+Wire Wire Line
+	6300 2900 5300 2900
+Wire Wire Line
+	5300 3100 7350 3100
+Wire Wire Line
+	7350 3300 6300 3300
+Wire Wire Line
+	6300 3300 6300 3200
+Wire Wire Line
+	6300 3200 5300 3200
+Wire Wire Line
+	5300 3400 7350 3400
+Wire Wire Line
+	6300 3600 6300 3500
+Wire Wire Line
+	6300 3500 5300 3500
+Wire Wire Line
+	5300 4200 5400 4200
+Connection ~ 5400 4200
+Wire Wire Line
+	5300 4300 6400 4300
+Wire Wire Line
+	6400 4300 6400 4000
+Connection ~ 5650 4300
+Text Label 5700 4000 0    39   ~ 0
+SCL
+Text Label 5700 4100 0    39   ~ 0
+SDA
+Text Label 5700 4300 0    39   ~ 0
++3V3
+Text Label 5700 3700 0    39   ~ 0
+CLK-
+Text Label 5700 3500 0    39   ~ 0
+CLK+
+Text Label 5700 3400 0    39   ~ 0
+D0-
+Text Label 5700 3200 0    39   ~ 0
+D0+
+Text Label 5700 3100 0    39   ~ 0
+D1-
+Text Label 5700 2900 0    39   ~ 0
+D1+
+Text Label 5700 2800 0    39   ~ 0
+D2-
+Text Label 5700 2600 0    39   ~ 0
+D2+
 $EndSCHEMATC
