File: electronics/ehdmifpc01/EAGLE/EHDMIFPC01.sch (EAGLE design)
At the start: 9 parts, among them J3 CONN-HDMI, J4 CONN-FFC-SFW15R

Commit message: Revision A, after assembling first batch of PCBs.
Changed lines of the file:
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@@
 <setting verticaltext="up"/>
 </settings>
-<grid distance="0.1" unitdist="inch" unit="inch" style="lines" multiple="1" display="no" altdistance="0.01" altunitdist="inch" altunit="inch"/>
+<grid distance="0.05" unitdist="inch" unit="inch" style="lines" multiple="1" display="no" altdistance="0.01" altunitdist="inch" altunit="inch"/>
 <layers>
 <layer number="1" name="Top" color="4" fill="1" visible="no" active="no"/>
@@
 <net name="CAM_0_N" class="0">
 <segment>
-<wire x1="129.54" y1="154.94" x2="154.305" y2="153.035" width="0.1524" layer="91"/>
+<wire x1="129.54" y1="154.94" x2="154.305" y2="155.575" width="0.1524" layer="91"/>
 <label x="139.065" y="153.035" size="1.778" layer="95"/>
 <pinref part="J4" gate="G$1" pin="2"/>
-<wire x1="154.305" y1="153.035" x2="154.305" y2="163.195" width="0.1524" layer="91"/>
+<wire x1="154.305" y1="155.575" x2="154.305" y2="163.195" width="0.1524" layer="91"/>
 <wire x1="203.2" y1="162.56" x2="154.305" y2="163.195" width="0.1524" layer="91"/>
 <pinref part="J3" gate="G$1" pin="1"/>
