File: electronics/emc01-drv/FPC-EMC01-1284.sch (EAGLE design)
At the start: 87 parts, among them J1 USB-MINIB-5PIN, J11 CONN-RECT-16PIN-2ROW, J12 CONN-RECT-16PIN-2ROW, J13 CONN-RECT-16PIN-2ROW, J14 CONN-RECT-16PIN-2ROW, J15 DNP, J16 ICSP, J2 CONN-MOLEX-MICROFIT-6PIN, J3 DNP, J4A MOT-X, J5A MOT-Y, J6A MOT-Z, J7A CONN-RECT-3PINJST_PH_2MM, J8A CONN-RECT-3PINJST_PH_2MM, J9A CONN-RECT-3PINJST_PH_2MM, Q2 2N7002PW, U1 IC-ATMEGA1284P-AU, U2 FT231XS, U3 IC-DRV8825, X1 16Mhz

Commit message: updated
Parts:
- removed STEPSTICK1, STEPSTICK3: STEPSTICK, FirePick:STEPSTICK
- added C21: 0.1 16V, SparkFun-Capacitors:CAP0805
- added C22, C23: 0.1, SparkFun-Capacitors:CAP0805
- added C24: 0.47 6.3V, SparkFun-Capacitors:CAP0805
- added R17, R18: 0.2, SparkFun-Resistors:RESISTOR0805-RES
- added R19: 20K, SparkFun-Resistors:RESISTOR0805-RES
- added SJ4, SJ5, SJ6: JUMPER, FirePick:JUMPER
- added U5: IC-DRV8825, FirePick:IC-DRV8825
- added VR2: 10K, adafruit:TRIMPOTTC33X
- C15: value 100uF -> 100 uF; device rcl:CPOL-USD -> rcl:CPOL-EUUD-6,3X7,7
- C17: value 100uF -> 0.01 50V; device rcl:CPOL-USD -> SparkFun-Capacitors:CAP0805
Connections:
- removed net !ENABLE: U3.!ENBL
- removed net +12V: C16.1, C18.1, C19.1, C28.+, U3.VMA, U3.VMB
- removed net DIR: U3.DIR
- removed net N$11: STEPSTICK1.!RESET!, STEPSTICK1.!SLEEP!
- removed net N$24: STEPSTICK3.!RESET!, STEPSTICK3.!SLEEP!
- removed net STEP: U3.STEP
- removed net Z2A: J6.3, J6A.3, STEPSTICK3.2A
- removed net Z2B: J6.4, J6A.4, STEPSTICK3.2B
- new net CP3: C17.1, U5.CP1
- new net CP4: C17.2, U5.CP2
- new net ISENA1: R18.2, U5.ISENA
- new net ISENB1: R17.2, U5.ISENB
- new net MOD2: SJ5.2, U5.MODE1
- new net MODE1: SJ4.2, U5.MODE0
- new net MODE3: SJ6.2, U5.MODE2
- new net N$7: R19.1, VR2.E
- new net N$8: J6.4, J6A.4, U5.AOUT2
- new net N$9: J6.3, J6A.3, U5.BOUT2
- new net V3P3OUT1: C24.1, R19.2, SJ4.1, SJ5.1, SJ6.1, U5.!RESET, U5.!SLEEP, U5.V3P3OUT
- new net VCP1: C21.2, U5.VCP
- new net VREF1: U5.AVREF, U5.BVREF, VR2.S
- net !XYZ_ENABLE: now also U3.!ENBL, U5.!ENBL; no longer STEPSTICK1.!ENABLE!, STEPSTICK3.!ENABLE!
- net +5V: no longer STEPSTICK1.MS1, STEPSTICK1.MS2, STEPSTICK1.MS3, STEPSTICK1.VDD, STEPSTICK3.MS1, STEPSTICK3.MS2, STEPSTICK3.MS3, STEPSTICK3.VDD
- net 12V: now also C16.1, C18.1, C19.1, C21.1, C22.1, C23.1, C28.+, U3.VMA, U3.VMB, U5.VMA, U5.VMB; no longer C17.+, STEPSTICK1.VMOT, STEPSTICK3.VMOT
- net GND: now also C22.2, C23.2, C24.2, R17.1, R18.1, U5.GND@1, U5.GND@2, U5.PPAD, U5.V1, U5.V10, U5.V11, U5.V12, U5.V13, U5.V14, U5.V15, U5.V16, U5.V17, U5.V18, U5.V19, U5.V2, U5.V20, U5.V21, U5.V3, U5.V4, U5.V5, U5.V6, U5.V7, U5.V8, U5.V9, VR2.A; no longer C17.-, STEPSTICK1.GND@1, STEPSTICK1.GND@2, STEPSTICK3.GND@1, STEPSTICK3.GND@2
- net X1A: no longer STEPSTICK1.1A
- net X1B: no longer STEPSTICK1.1B
- net X2A: no longer STEPSTICK1.2A
- net X2B: no longer STEPSTICK1.2B
- net X_DIR: no longer STEPSTICK1.DIR
- net X_STEP: no longer STEPSTICK1.STEP
- net Y_DIR: now also U3.DIR
- net Y_STEP: now also U3.STEP
- net Z1A: now also U5.BOUT1; no longer STEPSTICK3.1A
- net Z1B: now also U5.AOUT1; no longer STEPSTICK3.1B
- net Z_DIR: now also U5.DIR; no longer STEPSTICK3.DIR
- net Z_STEP: now also U5.STEP; no longer STEPSTICK3.STEP
Other:
- moved on the sheet: C15, J6, J6A

Commit message: New MCU Conversion
AT90 is hooked up in schematic
Parts:
- removed C10, C14, C6: 0.1uF, SparkFun-Capacitors:CAP0805
- removed C111, C17: 0.01 50V, SparkFun-Capacitors:CAP0805
- removed C12, C13: 47pF, SparkFun-Capacitors:CAP0805
- removed C15, C28: 100 uF, rcl:CPOL-EUUD-6,3X7,7
- removed C16, C21: 0.1 16V, SparkFun-Capacitors:CAP0805
- removed C18, C19, C22, C23: 0.1, SparkFun-Capacitors:CAP0805
- removed C20, C24: 0.47 6.3V, SparkFun-Capacitors:CAP0805
- removed FID1, FID2, FID3, FID4: FIDUCIAL1X2, SparkFun-Aesthetics:FIDUCIAL1X2
- removed J5, J6: (no value), !con-lstb:MA04-1
- removed J5A: MOT-Y, FirePick:CONN-RECT-4PINJST-PH-2MM
- removed J6A: MOT-Z, FirePick:CONN-RECT-4PINJST-PH-2MM
- removed Q2: 2N7002PW, SparkFun-DiscreteSemi:MOSFET-NCHANNEL2N7002PW
- removed R10, R11: 10k, SparkFun-Resistors:RESISTOR0805-RES
- removed R14, R15, R17, R18: 0.2, SparkFun-Resistors:RESISTOR0805-RES
- removed R16, R19: 20K, SparkFun-Resistors:RESISTOR0805-RES
- removed SJ1, SJ2, SJ3, SJ4, SJ5, SJ6: JUMPER, FirePick:JUMPER
- removed U3, U5: IC-DRV8825, FirePick:IC-DRV8825
- removed VR1, VR2: 10K, adafruit:TRIMPOTTC33X
- C2: value 4.7uF -> 1uF; device rcl:CPOL-USD -> SparkFun:CAP0805
- LOGO4: value LOGO-FIREPICK -> LOGO-FIREPICKLARGE; device FirePick:LOGO-FIREPICK -> FirePick:LOGO-FIREPICKLARGE
- LOGO6: value LOGO-CC-BY-SA -> LOGO-CC-BY-SALARGE; device FirePick:LOGO-CC-BY-SA -> FirePick:LOGO-CC-BY-SALARGE
- R8, R9: value 27 -> 22; device SparkFun-Resistors:RESISTOR0805-RES -> SparkFun:RESISTOR0805-RES
- U1: value IC-ATMEGA1284P-AU -> AT90USB1287-AU; device FirePick:IC-ATMEGA1284P-AU -> Atmel_By_element14_Batch_1-00:AT90USB1287-AU
- U2: value FT231XS -> PRTR5V0U4D; device SparkFun-DigitalIC:FT231XS -> printrbot:PRTR5V0U4D
- X1: value 16Mhz -> 20MHz
Connections:
- removed net CP1: C111.1, U3.CP1
- removed net CP2: C111.2, U3.CP2
- removed net CP3: C17.1, U5.CP1
- removed net CP4: C17.2, U5.CP2
- removed net DTR_3.3V: Q2.S, R10.1, U2.!DTR
- removed net ISENA: R15.2, U3.ISENA
- removed net ISENA1: R18.2, U5.ISENA
- removed net ISENB: R14.2, U3.ISENB
- removed net ISENB1: R17.2, U5.ISENB
- removed net MOD1: SJ2.2, U3.MODE1
- removed net MOD2: SJ5.2, U5.MODE1
- removed net MODE0: SJ1.2, U3.MODE0
- removed net MODE1: SJ4.2, U5.MODE0
- removed net MODE2: SJ3.2, U3.MODE2
- removed net MODE3: SJ6.2, U5.MODE2
- removed net N$23: R8.2, U2.USBDM
- removed net N$25: R9.2, U2.USBDP
- removed net N$3: R16.1, VR1.E
- removed net N$5: J5.2, J5A.2, U3.AOUT2
- removed net N$6: J5.1, J5A.1, U3.AOUT1
- removed net N$7: R19.1, VR2.E
- removed net N$8: J6.4, J6A.4, U5.AOUT2
- removed net N$9: J6.3, J6A.3, U5.BOUT2
- removed net V3P3OUT: C20.1, R16.2, SJ1.1, SJ2.1, SJ3.1, U3.!RESET, U3.!SLEEP, U3.V3P3OUT
- removed net V3P3OUT1: C24.1, R19.2, SJ4.1, SJ5.1, SJ6.1, U5.!RESET, U5.!SLEEP, U5.V3P3OUT
- removed net VCP: C16.2, U3.VCP
- removed net VCP1: C21.2, U5.VCP
- removed net VREF: U3.AVREF, U3.BVREF, VR1.S
- removed net VREF1: U5.AVREF, U5.BVREF, VR2.S
- removed net Z1A: J6.2, J6A.2, U5.BOUT1
- removed net Z1B: J6.1, J6A.1, U5.AOUT1
- new net SDCS: U1.PB0
- new net UCAP: C2.2, U1.UCAP
- new net VBUS: U1.VBUS, U2.VCC
- net !RESET: now also U1.~RESET; no longer U1.!RESET
- net !XYZ_ENABLE: now also U1.PC0; no longer U1.(PCINT30/OC2B/ICP)PD6, U3.!ENBL, U5.!ENBL
- net +5V: now also U1.UVCC, U1.VCC, U1.VCC_2; no longer C2.+, C6.1, R11.2, U1.VCC@1, U1.VCC@2, U1.VCC@3, U2.VCC
- net 12V: no longer C15.+, C16.1, C18.1, C19.1, C21.1, C22.1, C23.1, C28.+, U3.VMA, U3.VMB, U5.VMA, U5.VMB
- net 3.3V: no longer C10.1, Q2.G, R10.2, U2.!RESET, U2.3V3OUT, U2.VCCIO
- net AVR_RXD: now also U1.PD2; no longer U1.(PCINT24/RXD0/T3*)PD0
- net AVR_TXD: now also U1.PD3; no longer U1.(PCINT25/TXD0)PD1
- net D+: now also R9.2, U1.D+, U2.IO1; no longer C13.1, J1.D+, R9.1
- net D-: now also R8.2, U1.D-, U2.IO2; no longer C12.1, J1.D-, R8.1
- net DTR: no longer Q2.D, R11.1
- net GND: now also C2.1, U1.GND, U1.GND_2, U1.GND_3, U1.UGND, U2.GND; no longer C10.2, C12.2, C13.2, C14.2, C15.-, C18.2, C19.2, C2.-, C20.2, C22.2, C23.2, C24.2, C28.-, C6.2, R14.1, R15.1, R17.1, R18.1, U1.GND@1, U1.GND@2, U1.GND@3, U1.GND@4, U2.GND@16, U2.GND@6, U3.GND@1, U3.GND@2, U3.PPAD, U3.V1, U3.V10, U3.V11, U3.V12, U3.V13, U3.V14, U3.V15, U3.V16, U3.V17, U3.V18, U3.V19, U3.V2, U3.V20, U3.V21, U3.V3, U3.V4, U3.V5, U3.V6, U3.V7, U3.V8, U3.V9, U5.GND@1, U5.GND@2, U5.PPAD, U5.V1, U5.V10, U5.V11, U5.V12, U5.V13, U5.V14, U5.V15, U5.V16, U5.V17, U5.V18, U5.V19, U5.V2, U5.V20, U5.V21, U5.V3, U5.V4, U5.V5, U5.V6, U5.V7, U5.V8, U5.V9, VR1.A, VR2.A
- net MISO: now also U1.PB3; no longer U1.PB6(PCINT14/OC3A/MISO)
- net MOSI: now also U1.PB2; no longer U1.PB5(PCINT13/ICP3/MOSI)
- net N$1: now also J1.D-, R8.1; no longer J5.3, J5A.3, U3.BOUT2
- net N$2: now also J1.D+, R9.1; no longer J5.4, J5A.4, U3.BOUT1
- net RXD: no longer U2.RXD
- net RXLED: no longer U2.CBUS1
- net SCL: now also U1.PD0; no longer U1.(SCL/PCINT16)PC0
- net SCLK: now also U1.PB1; no longer U1.PB7(PCINT15/OC3B/SCK)
- net SDA: now also U1.PD1; no longer U1.(SDA/PCINT17)PC1
- net SPARE: now also U1.PE2; no longer U1.(PCINT26/RXD1/INT0)PD2
- net TOOL1_AIN: now also U1.PF0; no longer U1.PA0(ADC0/PCINT0)
- net TOOL1_DOUT: now also U1.PF1; no longer U1.PA1(ADC1/PCINT1)
- net TOOL1_ENABLE: now also U1.PB7; no longer U1.PB1(PCINT9/CLKO/T1)
- net TOOL2_AIN: now also U1.PF2; no longer U1.PA2(ADC2/PCINT2)
- net TOOL2_DOUT: now also U1.PF3; no longer U1.PA3(ADC3/PCINT3)
- net TOOL2_ENABLE: now also U1.PB6; no longer U1.PB0(PCINT8/XCK0/T0)
- net TOOL3_AIN: now also U1.PF5; no longer U1.PA5(ADC5/PCINT5)
- net TOOL3_DOUT: now also U1.PF4; no longer U1.PA4(ADC4/PCINT4)
- net TOOL3_ENABLE: now also U1.PB5; no longer U1.(TMS/PCINT19)PC3
- net TOOL4_AIN: now also U1.PF7; no longer U1.PA7(ADC7/PCINT7)
- net TOOL4_DOUT: now also U1.PF6; no longer U1.PA6(ADC6/PCINT6)
- net TOOL4_ENABLE: now also U1.PB4; no longer U1.(TCK/PCINT18)PC2
- net TOOL_DIR: now also U1.PA7; no longer U1.(OC2A/PCINT31)PD7
- net TOOL_STEP: now also U1.PA6; no longer U1.(TDO/PCINT20)PC4
- net TXD: no longer U2.TXD
- net TXLED: no longer U2.CBUS2
- net VUSB: no longer C14.1
- net X_DIR: now also U1.PA1; no longer U1.(TOSC1/PCINT22)PC6
- net X_STEP: now also U1.PA0; no longer U1.(TOSC2/PCINT23)PC7
- net X_STOP: now also U1.PE3; no longer U1.(TDI/PCINT21)PC5
- net Y_DIR: now also U1.PA3; no longer U1.PB3(PCINT11/OC0A/AIN1), U3.DIR
- net Y_STEP: now also U1.PA2; no longer U1.PB4(PCINT12/OC0B/SS), U3.STEP
- net Y_STOP: now also U1.PE4; no longer U1.PB2(PCINT10/INT2/AIN0)
- net Z_DIR: now also U1.PA5; no longer U1.(PCINT28/XCK1/OC1B)PD4, U5.DIR
- net Z_STEP: now also U1.PA4; no longer U1.(PCINT29/OC1A)PD5, U5.STEP
- net Z_STOP: now also U1.PE5; no longer U1.(PCINT27/TXD1/INT1)PD3
Other:
- note added: "ATMEL AT90USB1287-AU"
- note added: "Drawn by: NEIL JANSEN, DAYTON PIDHIRNEY"
- note added: "ESD"
- note added: "LEDS"
- note added: "USB-TO-TTL SERIAL"
- note removed: "ATMEL ATMEGA1284P-AU"
- note removed: "Drawn by: NEIL JANSEN"
- note removed: "FT231X USB-TO-TTL SERIAL"
- note removed: "Y AXIS STEPPER DRIVER"
- note removed: "Z AXIS STEPPER DRIVER"
- moved on the sheet: C11, C3, F1, J15, J16, J2, LED1, LED2, LED3, R12, R13, R3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
