File: electronics/EAT0001/EAT0001.brd (EAGLE design)
At the start: 29.2 x 33.2 mm, 35 parts, among them J1 CONN-RECT-16PIN-2ROWSIDE, J5 CONN-OSTTE1201X4, M1 FQD13N06LTM, U1 IC-DRV8825, U2 24AA014, U3 MIC5205

Commit message: Revision A, after assembling first batch of PCBs.
Parts:
- C2: value 1 -> 1uF 10V
- C28: value 100 uF -> 100 uF 25V
- C7, C8: value 0.1 -> 0.1uF 25V
- C9: value 0.47 6.3V -> 1 uF 10V
- R6, R7: value 0.2 -> 0.2 1% 1/4W
- R8: value 4.7K -> 4.7K 1%
- renumbered SJ1 to MS0, SJ2 to MS1, SJ3 to MS2
Connections:
- net 5V: now also U1.16, U1.17
- net V3P3OUT: no longer U1.16, U1.17
Routing:
- net 5V: track 12.9 -> 17.4 mm
- net V3P3OUT: track 28.0 -> 31.5 mm, vias 3 -> 2

Commit message: Updates to EAT0001 (Rev. A)
Parts:
- moved LOGO5 22.4 mm to (25.2, 20.2)
- moved LOGO4 0.80 mm to (13.4, 10.4)
Other:
- board text added: "Rev.A"
Changed lines of the file:
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@@
 <grid distance="0.2" unitdist="mm" unit="mm" style="lines" multiple="1" display="no" altdistance="0.025" altunitdist="inch" altunit="inch"/>
 <layers>
-<layer number="1" name="Top" color="4" fill="1" visible="yes" active="yes"/>
+<layer number="1" name="Top" color="4" fill="1" visible="no" active="yes"/>
 <layer number="2" name="PWR-5v" color="1" fill="3" visible="no" active="yes"/>
 <layer number="3" name="Route3" color="4" fill="3" visible="no" active="no"/>
@@
 <layer number="20" name="Dimension" color="15" fill="1" visible="yes" active="yes"/>
 <layer number="21" name="tPlace" color="7" fill="1" visible="no" active="yes"/>
-<layer number="22" name="bPlace" color="7" fill="1" visible="no" active="yes"/>
+<layer number="22" name="bPlace" color="7" fill="1" visible="yes" active="yes"/>
 <layer number="23" name="tOrigins" color="15" fill="1" visible="no" active="yes"/>
 <layer number="24" name="bOrigins" color="15" fill="1" visible="no" active="yes"/>
@@
 <layer number="30" name="bStop" color="7" fill="6" visible="no" active="yes"/>
 <layer number="31" name="tCream" color="7" fill="4" visible="no" active="yes"/>
-<layer number="32" name="bCream" color="7" fill="5" visible="no" active="yes"/>
+<layer number="32" name="bCream" color="7" fill="5" visible="yes" active="yes"/>
 <layer number="33" name="tFinish" color="6" fill="3" visible="no" active="yes"/>
 <layer number="34" name="bFinish" color="6" fill="6" visible="no" active="yes"/>
@@
 <wire x1="0" y1="5" x2="3.17" y2="5" width="0" layer="20"/>
 <wire x1="3.17" y1="5" x2="3.17" y2="0" width="0" layer="20"/>
-<text x="14" y="7.6" size="0.75" layer="21">P/N: EAT0001</text>
-<text x="14" y="8.6" size="0.75" layer="21">http://delta.firepick.org</text>
+<text x="13.6" y="8.2" size="0.75" layer="21">P/N: EAT0001</text>
+<text x="13.6" y="9.4" size="0.75" layer="21">http://delta.firepick.org</text>
 <text x="18.975734375" y="10.292890625" size="1" layer="22" rot="MR0">0</text>
 <text x="26" y="31" size="0.75" layer="22" rot="MR0">STEPPER MOTOR</text>
@@
 <vertex x="29.2" y="5"/>
 </polygon>
+<text x="13.6" y="7.2" size="0.75" layer="21">Rev.A</text>
 </plain>
 <attributes>
@@
 </element>
 <element name="C9" library="SparkFun-Capacitors" package="0805" value="1 uF 10V" x="12.3" y="13.9" smashed="yes" rot="R270">
-<attribute name="NAME" x="13.338" y="12.3255" size="1" layer="25"/>
+<attribute name="NAME" x="12.4745" y="16.138" size="1" layer="25" rot="R90"/>
 <attribute name="VALUE" x="10.903" y="14.916" size="0.4064" layer="27" rot="R270"/>
 </element>
@@
 <element name="FID3" library="SparkFun-Aesthetics" package="FIDUCIAL-1X2" value="FIDUCIAL1X2" x="1.6" y="31.4"/>
 <element name="FID4" library="SparkFun-Aesthetics" package="FIDUCIAL-1X2" value="FIDUCIAL1X2" x="24.6" y="7.2" rot="R90"/>
-<element name="LOGO4" library="FirePick" package="LOGO-FIREPICK-MEDIUM" value="LOGO-FIREPICKMEDIUM" x="13.4" y="9.6"/>
-<element name="LOGO5" library="FirePick" package="LOGO-OSHW-SMALL" value="LOGO-OSHWSMALL" x="2.8" y="21" rot="MR0"/>
+<element name="LOGO4" library="FirePick" package="LOGO-FIREPICK-MEDIUM" value="LOGO-FIREPICKMEDIUM" x="13.4" y="10.4"/>
+<element name="LOGO5" library="FirePick" package="LOGO-OSHW-SMALL" value="LOGO-OSHWSMALL" x="25.2" y="20.2" rot="MR0"/>
 <element name="LOGO6" library="FirePick" package="LOGO-CC-BY-SA-MEDIUM" value="LOGO-CC-BY-SAMEDIUM" x="23" y="16.4" rot="MR0"/>
 <element name="R4" library="SparkFun-Resistors" package="0805" value="10k" x="8.4" y="7" smashed="yes" rot="MR0">
@@
 <wire x1="15" y1="13.6" x2="16" y2="13.6" width="0.3" layer="16"/>
 <wire x1="16" y1="13.6" x2="17.4869" y2="12.1131" width="0.3" layer="16"/>
-<wire x1="15" y1="13.6" x2="16.8" y2="15.4" width="0.254" layer="15"/>
-<wire x1="16.8" y1="15.4" x2="17.4" y2="15.4" width="0.254" layer="15"/>
+<wire x1="15" y1="13.6" x2="16.8" y2="15.4" width="0.3" layer="15"/>
+<wire x1="16.8" y1="15.4" x2="17.4" y2="15.4" width="0.3" layer="15"/>
 </signal>
 </signals>

Commit message: minor cosmetic and refdes updates
Parts:
- renumbered M1 to Q1
Changed lines of the file:
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@@
 <layer number="19" name="Unrouted" color="6" fill="1" visible="yes" active="yes"/>
 <layer number="20" name="Dimension" color="15" fill="1" visible="yes" active="yes"/>
-<layer number="21" name="tPlace" color="7" fill="1" visible="no" active="yes"/>
-<layer number="22" name="bPlace" color="7" fill="1" visible="yes" active="yes"/>
+<layer number="21" name="tPlace" color="7" fill="1" visible="yes" active="yes"/>
+<layer number="22" name="bPlace" color="7" fill="1" visible="no" active="yes"/>
 <layer number="23" name="tOrigins" color="15" fill="1" visible="no" active="yes"/>
 <layer number="24" name="bOrigins" color="15" fill="1" visible="no" active="yes"/>
-<layer number="25" name="tNames" color="7" fill="1" visible="no" active="yes"/>
+<layer number="25" name="tNames" color="7" fill="1" visible="yes" active="yes"/>
 <layer number="26" name="bNames" color="7" fill="1" visible="no" active="yes"/>
 <layer number="27" name="tValues" color="7" fill="1" visible="no" active="yes"/>
@@
 <layer number="29" name="tStop" color="7" fill="3" visible="no" active="yes"/>
 <layer number="30" name="bStop" color="7" fill="6" visible="no" active="yes"/>
-<layer number="31" name="tCream" color="7" fill="4" visible="no" active="yes"/>
-<layer number="32" name="bCream" color="7" fill="5" visible="yes" active="yes"/>
+<layer number="31" name="tCream" color="7" fill="4" visible="yes" active="yes"/>
+<layer number="32" name="bCream" color="7" fill="5" visible="no" active="yes"/>
 <layer number="33" name="tFinish" color="6" fill="3" visible="no" active="yes"/>
 <layer number="34" name="bFinish" color="6" fill="6" visible="no" active="yes"/>
@@
 <attribute name="NAME" x="6.207" y="10.632" size="1.016" layer="26" ratio="10" rot="MR0"/>
 </element>
-<element name="M1" library="SparkFun" package="DPAK" value="FQD13N06LTM" x="7.6" y="20.46" smashed="yes">
+<element name="Q1" library="SparkFun" package="DPAK" value="FQD13N06LTM" x="7.6" y="20.46" smashed="yes">
 <attribute name="NAME" x="6.758" y="13.883" size="1" layer="25"/>
 <attribute name="VALUE" x="11.537" y="16.758" size="0.4064" layer="27" rot="R90"/>
@@
 <signal name="GND">
 <contactref element="U2" pad="2"/>
-<contactref element="M1" pad="3"/>
+<contactref element="Q1" pad="3"/>
 <contactref element="C28" pad="-"/>
 <contactref element="U1" pad="PAD"/>
@@
 <signal name="DOUT">
 <contactref element="J1" pad="14"/>
-<contactref element="M1" pad="1"/>
+<contactref element="Q1" pad="1"/>
 <contactref element="R3" pad="2"/>
 <wire x1="5.32" y1="15.15" x2="5.32" y2="13.32" width="0.5" layer="1"/>
@@
 </signal>
 <signal name="HOTBED-GND" class="2">
-<contactref element="M1" pad="4"/>
+<contactref element="Q1" pad="4"/>
 <polygon width="1" layer="16" isolate="0.5" orphans="yes">
 <vertex x="9.6" y="24.4"/>

Commit message: Moving STL's over here
Parts:
- moved LOGO1 8.07 mm to (6.40, 26.4)
- moved LOGO6 3.00 mm to (25.4, 14.6)
- moved LOGO4 0.45 mm to (13.0, 10.6)
- moved R4 0.05 mm to (8.35, 7.00), turned to 180 degrees
Connections:
- removed net 3.3V: R4.1, R5.1
- net 5V: now also R4.1, R5.1
Routing:
- net 3.3V: track 14.9 -> 0.00 mm, vias 2 -> 0
- net 5V: track 17.4 -> 26.3 mm
Other:
- board text added: "THRM"
- board text removed: "THRMSTR"
