File: electronics/EAT0001/EAT0001.sch (EAGLE design)
At the start: 35 parts, among them J1 CONN-RECT-16PIN-2ROWSIDE, J5 CONN-OSTTE1201X4, M1 FQD13N06LTM, U1 IC-DRV8825, U2 24AA014, U3 MIC5205

Commit message: Revision A, after assembling first batch of PCBs.
Parts:
- C2: value 1 -> 1uF 10V
- C28: value 100 uF -> 100 uF 25V
- C7, C8: value 0.1 -> 0.1uF 25V
- C9: value 0.47 6.3V -> 1 uF 10V
- R6, R7: value 0.2 -> 0.2 1% 1/4W
- R8: value 4.7K -> 4.7K 1%
- renumbered SJ1 to MS0, SJ2 to MS1, SJ3 to MS2
Connections:
- net 5V: now also U1.!RESET, U1.!SLEEP
- net V3P3OUT: no longer U1.!RESET, U1.!SLEEP
Other:
- note added: "Rev. A: * Remove wires from /SLEEP and /RESET to V3P3OUT. * Add wire from /SLEEP and /RESET to +5V net"
- note added: "TODO: Add LED to /ENABLE pin"
- moved on the sheet: C28, C7, C8, R6, R7

Commit message: Updates to EAT0001 (Rev. A)
Other:
- note added: "Rev A"
- note removed: "v0.1"
Changed lines of the file:
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@@
 <text x="289.56" y="20.32" size="1.778" layer="94" ratio="15">Drawn by: NEIL JANSEN</text>
 <text x="289.56" y="16.51" size="1.778" layer="94" ratio="15">Checked  by:</text>
-<text x="374.65" y="5.08" size="2.54" layer="94" ratio="10">v0.1</text>
+<text x="290.83" y="7.62" size="2.54" layer="94" ratio="10">Rev A</text>
 <wire x1="5.715" y1="28.575" x2="288.29" y2="28.575" width="0.3048" layer="94"/>
 <wire x1="288.29" y1="28.575" x2="288.29" y2="3.81" width="0.3048" layer="94"/>

Commit message: minor cosmetic and refdes updates
Parts:
- renumbered M1 to Q1
Changed lines of the file:
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@@
 <part name="GND3" library="supply1" deviceset="GND" device=""/>
 <part name="GND69" library="SparkFun" deviceset="GND" device=""/>
-<part name="M1" library="SparkFun" deviceset="MOSFET-NCHANNEL" device="FDD8580" value="FQD13N06LTM"/>
+<part name="Q1" library="SparkFun" deviceset="MOSFET-NCHANNEL" device="FDD8580" value="FQD13N06LTM"/>
 <part name="GND70" library="SparkFun" deviceset="GND" device=""/>
 <part name="C28" library="rcl" deviceset="CPOL-EU" device="UD-6,3X7,7" value="100 uF 25V"/>
@@
 <instance part="GND3" gate="1" x="55.88" y="63.5"/>
 <instance part="GND69" gate="1" x="241.3" y="66.04"/>
-<instance part="M1" gate="G$1" x="241.3" y="81.28"/>
+<instance part="Q1" gate="G$1" x="241.3" y="81.28"/>
 <instance part="GND70" gate="1" x="231.14" y="66.04"/>
 <instance part="C28" gate="G$1" x="160.02" y="152.4"/>
@@
 <wire x1="241.3" y1="76.2" x2="241.3" y2="68.58" width="0.1524" layer="91"/>
 <pinref part="GND69" gate="1" pin="GND"/>
-<pinref part="M1" gate="G$1" pin="S"/>
+<pinref part="Q1" gate="G$1" pin="S"/>
 </segment>
 <segment>
@@
 <wire x1="233.68" y1="81.28" x2="231.14" y2="81.28" width="0.1524" layer="91"/>
 <label x="215.9" y="81.28" size="1.778" layer="95"/>
-<pinref part="M1" gate="G$1" pin="G"/>
+<pinref part="Q1" gate="G$1" pin="G"/>
 <pinref part="R3" gate="G$1" pin="2"/>
 <wire x1="231.14" y1="81.28" x2="215.9" y2="81.28" width="0.1524" layer="91"/>
@@
 <net name="HOTBED-GND" class="2">
 <segment>
-<pinref part="M1" gate="G$1" pin="D"/>
+<pinref part="Q1" gate="G$1" pin="D"/>
 <wire x1="261.62" y1="88.9" x2="241.3" y2="88.9" width="0.1524" layer="91"/>
 <wire x1="241.3" y1="88.9" x2="241.3" y2="86.36" width="0.1524" layer="91"/>

Commit message: Moving STL's over here
Connections:
- removed net 3.3V: R4.1, R5.1
- net 5V: now also R4.1, R5.1
Other:
- note added: "Rev B"
- note added: "Rev. B: * Silkscreen and cosmetic updates * Fix pullups on U2 A0/A1 to +5V net"
- note removed: "Rev A"
- note removed: "TODO: Add LED to /ENABLE pin"
- note removed: "TODO: For beefier version, change MOSFET to 060N06"
- moved on the sheet: C111, C28, C5, C7, C8, C9, J1, J5, MS0, MS1, MS2, R1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
