File: electronics/emc02/EMC02.brd (EAGLE design)
At the start: 150 x 129.9 mm, 117 parts, among them IC1 74ACT244DW, IC2 74ACT244DW, IC3 INA168, J11 CONN-RECT-16PIN-2ROW, J12 CONN-RECT-16PIN-2ROW, J13 CONN-RECT-16PIN-2ROW, J14 CONN-RECT-16PIN-2ROW, J15 DNP, J16 MA18-1, J22 OSTTH050160, J23 ICSP/SPI, J4A MOT-X, J5A MOT-Y, J6A MOT-Z, Q1 BSS138, Q2 BSS138, Q3 BSS138

Commit message: Moving STL's over here
Parts:
- added C10, C11, C8, C9: 100uF, rcl:PANASONIC_D
- added C5, C6, C7: 0.1u, SparkFun-Capacitors:0805
- added J21: (no value), !con-lstb:MA09-1
- added J22A: OSTTH050160, FirePick:CONN-OSTTH050160
- added Q4: BSS138, SparkFun-DiscreteSemi:SOT23
- added R35: 4.7K 0.1%, SparkFun-Resistors:0805
- added R36, R46, R47: 10K, SparkFun-Resistors:0805
- added R37: 4.7k 0.1%, SparkFun-Resistors:0805
- added R44: 100K, SparkFun-Resistors:0805
- added R45: 10k 0.1%, SparkFun-Resistors:0805
- added U$25: TIN-WHISKERSTSTOP, !tin-whiskers:TIN-WHISKERS-TSTOP
- FAN1, FAN2: value (none) -> 22232031
- FID1, FID2, FID3, FID4, FID5, FID6, FID7: value FIDUCIAL1X2 -> FIDUCIAL; device SparkFun-Aesthetics:FIDUCIAL-1X2 -> FirePick:FIDUCIAL
- J1, J17, J2, J24, J25, J26, J27, J28, J29, J3, J30: value (none) -> CONN-0.1-S-1X3
- J16: value MA18-1 -> CONN-0.1-S-1x18
- J18, J19, J20: value (none) -> CONN-0.1-S-2X3
- J22: value OSTTH050160 -> OSTOP050000; device FirePick:CONN-OSTTH050160 -> FirePick:CONN-OSTOP050000
- J31: value (none) -> CONN-0.1-S-1X2
- J4, J5, J6: value (none) -> CONN-0.1-RA-1X4
- J7, J8, J9: value (none) -> CONN-0.1-RA-1X3
- J7A, J8A, J9A: value (none) -> CONN-RECT-3PINJST_PH_2MM
- LED1: value Green -> AMBER
- LED2: value Red -> AMBER
- LED3: value Yellow -> AMBER
- R34: value RESISTOR-KELVIN -> 1.0 mOhm
- moved IC3 223.4 mm to (51.2, 112.7), turned to 270 degrees
- moved FAN2 214.2 mm to (140.2, 55.7), turned to 240 degrees
- moved J22 100.2 mm to (75.0, 126.0)
- moved R1 99.6 mm to (63.2, 108.5)
- moved ARDUINO 99.2 mm to (48.2, -5.40)
- moved C1 99.2 mm to (81.5, 56.0)
- moved C15 99.2 mm to (81.3, 108.3)
- moved C16 99.2 mm to (33.4, 52.1)
- moved C17 99.2 mm to (111.8, 43.1)
- moved C2 99.2 mm to (82.2, 36.2)
- moved C3 99.2 mm to (119.2, 67.2)
- moved C4 99.2 mm to (29.2, 61.2)
- moved D1 99.2 mm to (77.8, 7.45)
- moved FID1 99.2 mm to (9.00, 65.0)
- moved FID2 99.2 mm to (141.0, 65.0)
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Connections:
- removed net V+: IC3.5
- removed net V-: IC3.2
- new net 20_SDA: ARDUINO.20, J21.3
- new net 21_SCL: ARDUINO.21, J21.2
- new net FAN2_PWM: ARDUINO.10, Q4.1, R46.2
- new net FAN2_TACH: ARDUINO.11, FAN2.3, R47.2
- new net ISENSE: ARDUINO.A8, C6.1, IC3.1, R44.2
- new net N$17: C7.1, IC3.3, IC3.5, R34.I1, R35.2
- new net N$18: IC3.4, R34.I2
- new net N$3: J22.1, R34.V1
- new net RX1: ARDUINO.19, J21.4
- new net RX2: ARDUINO.17, J21.6
- new net RX3: ARDUINO.15, J21.8
- new net TX1: ARDUINO.18, J21.5
- new net TX2: ARDUINO.16, J21.7
- new net TX3: ARDUINO.14, J21.9
- new net VSENSE: ARDUINO.A1, C5.1, R37.2, R45.1
- net !PS_ON_BUF: now also R36.2
- net !TOOL4_EN_BUF: now also ARDUINO.34; no longer ARDUINO.19
- net 12V: now also C10.+, C11.+, C8.+, C9.+, R34.V2; no longer ARDUINO.VIN, J22.1
- net GND: now also C10.-, C11.-, C5.2, C6.2, C7.2, C8.-, C9.-, IC3.2, J21.1, Q4.2, R36.1, R37.1, R44.1; no longer FAN2.1
- net IOREF: now also R46.1, R47.1
- net N$1: now also R35.1, R45.2; no longer FAN1.3
- net N$2: now also FAN2.1, Q4.3; no longer FAN2.3
- net TOOL4_DOUT_BUF: now also ARDUINO.26; no longer ARDUINO.18
Routing:
- net VSENSE: track 0.00 -> 85.8 mm, vias 0 -> 3
- net FAN2_PWM: track 0.00 -> 62.1 mm, vias 0 -> 2
- net ISENSE: track 0.00 -> 60.1 mm, vias 0 -> 3
- net FAN2_TACH: track 0.00 -> 56.8 mm
- net IOREF: track 116.0 -> 137.0 mm, vias 0 -> 2
- net N$17: track 0.00 -> 20.2 mm
- net TOOL4_DOUT_BUF: track 36.3 -> 52.6 mm, vias 2 -> 3
- net N$18: track 0.00 -> 10.4 mm
- net +5V: track 524.0 -> 514.1 mm
- net 12V: track 359.1 -> 365.9 mm, vias 0 -> 3
- net !PS_ON_BUF: track 24.7 -> 30.5 mm
- net N$3: track 0.00 -> 5.51 mm
- net N$2: track 0.00 -> 5.36 mm
- net RX2: track 0.00 -> 3.04 mm
- net RX1: track 0.00 -> 3.04 mm
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Other:
- board text added: "20_SDA"
- board text added: "21_SCL"
- board text added: "FAN1"
- board text added: "FAN2"
- board text added: "P/N: EMC02 Rev B"
- board text added: "PS-ON"
- board text added: "RX1"
- board text added: "RX2"
- board text added: "RX3"
- board text added: "STDBY"
- board text added: "TX1"
- board text added: "TX2"
- board text added: "TX3"
- board text removed: "FAN"
- board text removed: "P/N: EMC02 Rev A"
- board text removed: "PS_ON"
