File: electronics/emc02/EMC02.sch (EAGLE design)
At the start: 117 parts, among them IC1 74ACT244DW, IC2 74ACT244DW, IC3 INA168, J11 CONN-RECT-16PIN-2ROW, J12 CONN-RECT-16PIN-2ROW, J13 CONN-RECT-16PIN-2ROW, J14 CONN-RECT-16PIN-2ROW, J15 DNP, J16 MA18-1, J22 OSTTH050160, J23 ICSP/SPI, J4A MOT-X, J5A MOT-Y, J6A MOT-Z, J7A CONN-RECT-3PINJST_PH_2MM, J8A CONN-RECT-3PINJST_PH_2MM, J9A CONN-RECT-3PINJST_PH_2MM, Q1 BSS138, Q2 BSS138, Q3 BSS138

Commit message: Moving STL's over here
Parts:
- added C10, C11, C8, C9: 100uF, rcl:CPOL-USD
- added C5, C6, C7: 0.1u, SparkFun-Capacitors:CAP0805
- added J21: (no value), !con-lstb:MA09-1
- added J22A: OSTTH050160, FirePick:CONN-OSTTH050160
- added Q4: BSS138, SparkFun-DiscreteSemi:MOSFET-NCHANNELBSS138
- added R35: 4.7K 0.1%, SparkFun-Resistors:RESISTOR0805-RES
- added R36, R46, R47: 10K, SparkFun-Resistors:RESISTOR0805-RES
- added R37: 4.7k 0.1%, SparkFun-Resistors:RESISTOR0805-RES
- added R44: 100K, SparkFun-Resistors:RESISTOR0805-RES
- added R45: 10k 0.1%, SparkFun-Resistors:RESISTOR0805-RES
- added U$25: TIN-WHISKERSTSTOP, !tin-whiskers:TIN-WHISKERSTSTOP
- ARDUINO: PARTNO (none) -> CONN-0.1-ARD-2560
- C1, C2, C4: PARTNO (none) -> CC0805ZRY5V9BB104
- C15, C16, C17, C3: PARTNO (none) -> 25TXV100M6.3X8
- D1: PARTNO (none) -> 1N4148W-7-F
- FAN1, FAN2: value (none) -> 22232031; PARTNO (none) -> 22232031
- FID1, FID2, FID3, FID4, FID5, FID6, FID7: value FIDUCIAL1X2 -> FIDUCIAL; device SparkFun-Aesthetics:FIDUCIAL1X2 -> FirePick:FIDUCIAL; BOM (none) -> EXCLUDE
- IC1, IC2: PARTNO (none) -> 74ACT244SCX
- IC3: DNP (none) -> T; PARTNO (none) -> INA168NA/3K
- J1, J17, J2, J24, J25, J26, J27, J28, J29, J3, J30: value (none) -> CONN-0.1-S-1X3; PARTNO (none) -> CONN-0.1-S-1X3
- J10, J15, J23, J4A, J5A, J6A, J7A, J8A, J9A, R38, R39, TP2, TP3, TP4, TP5: DNP (none) -> T
- J11, J12, J13, J14, STEPSTICK1, STEPSTICK2, STEPSTICK3: PARTNO (none) -> PPPC081LFBN-RC
- J16: value MA18-1 -> CONN-0.1-S-1x18; DNP (none) -> T
- J18, J19, J20: value (none) -> CONN-0.1-S-2X3; PARTNO (none) -> CONN-0.1-S-2X3
- J22: value OSTTH050160 -> OSTOP050000; device FirePick:CONN-OSTTH050160 -> FirePick:CONN-OSTOP050000; PARTNO (none) -> OSTOP240000
- J31: value (none) -> CONN-0.1-S-1X2; PARTNO (none) -> CONN-0.1-S-1X2
- J4, J5, J6: value (none) -> CONN-0.1-RA-1X4; PARTNO (none) -> CONN-0.1-RA-1X4
- J7, J8, J9: value (none) -> CONN-0.1-RA-1X3; PARTNO (none) -> CONN-0.1-RA-1X3
- LED1: value Green -> AMBER; PARTNO (none) -> LTST-C150AKT
- LED2: value Red -> AMBER; PARTNO (none) -> LTST-C150AKT
- LED3: value Yellow -> AMBER; PARTNO (none) -> LTST-C150AKT
- LOGO1, LOGO2, LOGO3, LOGO4, LOGO5, LOGO6: BOM (none) -> EXCLUDE
- Q1, Q2, Q3: PARTNO (none) -> BSS138
- R1, R29, R6, R7: PARTNO (none) -> RC0805FR-07100KL
- R10, R11, R14, R15, R28: PARTNO (none) -> RC0805FR-074K7L
- R12, R13, R16, R18, R2, R25, R26, R27, R30, R31, R32, R33, R40, R41, R42, R43, R8, R9: PARTNO (none) -> RC0805FR-0710KL
- R17, R19, R20, R21, R22, R23, R24: PARTNO (none) -> RC0805FR-0720KL
- R3, R4, R5: PARTNO (none) -> RC0805FR-071KL
- R34: value RESISTOR-KELVIN -> 1.0 mOhm; PARTNO (none) -> LVK25R001FER
- S1: PARTNO (none) -> SWITCH TACTILE SPST-NO 0.05A 12V
Connections:
- new net 20_SDA: ARDUINO.20(SDA), J21.3
- new net 21_SCL: ARDUINO.21(SCL), J21.2
- new net FAN2_PWM: ARDUINO.10, Q4.G, R46.2
- new net FAN2_TACH: ARDUINO.11, FAN2.3, R47.2
- new net ISENSE: ARDUINO.A8, C6.1, IC3.OUT, R44.2
- new net N$17: C7.1, IC3.IN+, IC3.V+, R34.I1, R35.2
- new net N$18: IC3.IN-, R34.I2
- new net N$3: J22.1, R34.V1
- new net RX1: ARDUINO.19(RX1), J21.4
- new net RX2: ARDUINO.17(RX2), J21.6
- new net RX3: ARDUINO.15(RX3), J21.8
- new net TX1: ARDUINO.18(TX1), J21.5
- new net TX2: ARDUINO.16(TX2), J21.7
- new net TX3: ARDUINO.14(TX3), J21.9
- new net VSENSE: ARDUINO.A1(TX0), C5.1, R37.2, R45.1
- net !PS_ON_BUF: now also R36.2
- net !TOOL4_EN_BUF: now also ARDUINO.34; no longer ARDUINO.19(RX1)
- net 12V: now also C10.+, C11.+, C8.+, C9.+, R34.V2; no longer ARDUINO.VIN, J22.1
- net GND: now also C10.-, C11.-, C5.2, C6.2, C7.2, C8.-, C9.-, IC3.V-, J21.1, Q4.S, R36.1, R37.1, R44.1; no longer FAN2.1
- net IOREF: now also R46.1, R47.1
- net N$1: now also R35.1, R45.2; no longer FAN1.3
- net N$2: now also FAN2.1, Q4.D; no longer FAN2.3
- net TOOL4_DOUT_BUF: now also ARDUINO.26; no longer ARDUINO.18(TX1)
Other:
- note added: "* NOTE: THIS IS A 2-PIECE TERMINAL STRIP. - THE OSTOP IS THE MALE PIN HEADER - THE OSTTH IS THE PLUG-ON SCREW TERMINAL"
- note added: "AVR JTAG"
- note added: "C8-C11 ARE OPTIONAL (DNP)"
- note added: "Isense Vout=(Is)(Rs)(200uA/V)(RL) = 15A * 0.001 ohm * 0.0002 A/V * RL"
- note added: "NOTE: FAN1 IS INTENDED FOR END EFFECTOR (CONSTANT ON) FAN2 IS INTENDED FOR PLA COOLING (SWITCHED)"
- note added: "NOTE: FOR MEGA 2560, - PIN 50 CONNECTED TO 'MISO - PIN 51 CONNECTED TO MOSI - PIN 52 CONNECTED TO SCK - PIN 53 CONNECTED TO SS"
- note added: "Revision B"
- note added: "Revision B: Added R36,R45,C7. Unconnected Arduino VIN to +12V. Fixed PCB routing issue. Moved TOOL4_DOUT_BUF and !TOOL4_EN_BUF! from 18/19 to"
- note added: "SERIAL"
- note added: "SPI BUS"
- note added: "TODO: INSTALL FERRITE BEAD ON ISENSE?"
- note removed: "* Add current & voltage monitoring circuits"
- note removed: "AVR JTAG/GPIO"
- note removed: "ICSP"
- note removed: "Revision --"
- note removed: "Revision A"
- note removed: "TODO: ** ADD FIDUCIALS"
- note removed: "TODO: PWM CONTROL FAN #2"
- note removed: "TODO: TACH ON 1 OR BOTH FANS"
- moved on the sheet: C1, C2, C3, C4, FAN1, FAN2, IC1P, IC2P, IC3, J1, J10, J15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
