File: electronics/eopto01/EAGLE/EOPTO01.brd (EAGLE design)
At the start: 35.3 x 12 mm, 13 parts, among them J1 CONN-RECT-3PINJST_PH_2MM, Q1 BC849

Commit message: Revision A, after assembling first batch of PCBs.
Parts:
- removed Q1: BC849, transistor:SOT23
- added Q2: BSS138, SparkFun-DiscreteSemi:SOT23
- R1: value (none) -> 120
- R2: value (none) -> 10k
- R3: value (none) -> 1k
Connections:
- net GND: now also Q2.2; no longer Q1.2
- net N$2: now also Q2.3; no longer Q1.3
- net OPTO_OUT: now also Q2.1; no longer Q1.1
Routing:
- net OPTO_OUT: track 24.8 -> 25.6 mm
Other:
- board text added: "+"
- board text added: "D"
- board text added: "E"
Changed lines of the file:
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@@
 <grid distance="0.2" unitdist="mm" unit="mm" style="lines" multiple="1" display="no" altdistance="0.025" altunitdist="inch" altunit="inch"/>
 <layers>
-<layer number="1" name="Top" color="4" fill="1" visible="no" active="yes"/>
+<layer number="1" name="Top" color="4" fill="1" visible="yes" active="yes"/>
 <layer number="2" name="Route2" color="1" fill="3" visible="no" active="no"/>
 <layer number="3" name="Route3" color="4" fill="3" visible="no" active="no"/>
 <layer number="14" name="Route14" color="1" fill="6" visible="no" active="no"/>
 <layer number="15" name="Route15" color="4" fill="6" visible="no" active="no"/>
-<layer number="16" name="Bottom" color="1" fill="1" visible="no" active="yes"/>
+<layer number="16" name="Bottom" color="1" fill="1" visible="yes" active="yes"/>
 <layer number="17" name="Pads" color="2" fill="1" visible="yes" active="yes"/>
 <layer number="18" name="Vias" color="2" fill="1" visible="yes" active="yes"/>
 <layer number="19" name="Unrouted" color="6" fill="1" visible="yes" active="yes"/>
 <layer number="20" name="Dimension" color="15" fill="1" visible="yes" active="yes"/>
-<layer number="21" name="tPlace" color="7" fill="1" visible="no" active="yes"/>
-<layer number="22" name="bPlace" color="7" fill="1" visible="yes" active="yes"/>
+<layer number="21" name="tPlace" color="7" fill="1" visible="yes" active="yes"/>
+<layer number="22" name="bPlace" color="7" fill="1" visible="no" active="yes"/>
 <layer number="23" name="tOrigins" color="15" fill="1" visible="yes" active="yes"/>
-<layer number="24" name="bOrigins" color="15" fill="1" visible="yes" active="yes"/>
-<layer number="25" name="tNames" color="7" fill="1" visible="no" active="yes"/>
-<layer number="26" name="bNames" color="7" fill="1" visible="yes" active="yes"/>
+<layer number="24" name="bOrigins" color="15" fill="1" visible="no" active="yes"/>
+<layer number="25" name="tNames" color="7" fill="1" visible="yes" active="yes"/>
+<layer number="26" name="bNames" color="7" fill="1" visible="no" active="yes"/>
 <layer number="27" name="tValues" color="7" fill="1" visible="no" active="yes"/>
 <layer number="28" name="bValues" color="7" fill="1" visible="no" active="yes"/>
@@
 <text x="25.4" y="7.6" size="1" layer="22" ratio="15" rot="MR0">http://delta.firepick.org</text>
 <text x="30.8" y="1.2" size="1" layer="22" ratio="15" rot="MR90">P/N: EOPTO01</text>
+<text x="7" y="5.8" size="1" layer="21">+</text>
+<text x="14.6" y="1.4" size="1" layer="21">+</text>
+<text x="7.2" y="1.4" size="1" layer="21">E</text>
+<text x="14.8" y="5.8" size="1" layer="21">D</text>
 </plain>
 <attributes>
@@
 </element>
 <element name="J2" library="!con-lstb" package="MA03-1" value="" x="33.67" y="6" smashed="yes" rot="R90"/>
-<element name="R1" library="SparkFun-Resistors" package="0805" value="" x="5.8" y="9.6" smashed="yes" rot="R270">
+<element name="R1" library="SparkFun-Resistors" package="0805" value="120" x="5.8" y="9.6" smashed="yes" rot="R270">
 <attribute name="NAME" x="2.808" y="10.1955" size="1" layer="25"/>
 <attribute name="VALUE" x="4.403" y="10.616" size="0.4064" layer="27" rot="R270"/>
 </element>
-<element name="R2" library="SparkFun-Resistors" package="0805" value="" x="17.2" y="9.6" smashed="yes" rot="R90">
+<element name="R2" library="SparkFun-Resistors" package="0805" value="10k" x="17.2" y="9.6" smashed="yes" rot="R90">
 <attribute name="NAME" x="18.238" y="10.4255" size="1" layer="25"/>
 <attribute name="VALUE" x="18.597" y="8.584" size="0.4064" layer="27" rot="R90"/>
 </element>
-<element name="R3" library="SparkFun-Resistors" package="0805" value="" x="8.6" y="9.6" smashed="yes" rot="R90">
+<element name="R3" library="SparkFun-Resistors" package="0805" value="1k" x="8.6" y="9.6" smashed="yes" rot="R90">
 <attribute name="NAME" x="9.448" y="10.2155" size="1" layer="25"/>
 <attribute name="VALUE" x="9.997" y="8.584" size="0.4064" layer="27" rot="R90"/>
@@
 <attribute name="NAME" x="11.861" y="10.117" size="1" layer="25"/>
 <attribute name="VALUE" x="11.734" y="6.942" size="0.4064" layer="27"/>
-</element>
-<element name="Q1" library="transistor" package="SOT23" value="BC849" x="21.84" y="9.6" smashed="yes" rot="R90">
-<attribute name="NAME" x="23.695" y="9.865" size="1.27" layer="25"/>
 </element>
 <element name="OPTO1" library="FirePick" package="TCST2013" value="TCST2103" x="12.75" y="4" smashed="yes">
@@
 <element name="LOGO5" library="FirePick" package="LOGO-OSHW-SMALL" value="LOGO-OSHWSMALL" x="14.02" y="2.98" rot="MR0"/>
 <element name="LOGO6" library="FirePick" package="LOGO-CC-BY-SA-MEDIUM" value="LOGO-CC-BY-SAMEDIUM" x="10.61" y="8" rot="MR0"/>
+<element name="Q2" library="SparkFun-DiscreteSemi" package="SOT23" value="BSS138" x="21.4" y="9.6" rot="R90">
+<attribute name="PROD_ID" value="TRANS-00830" x="21.4" y="9.6" size="1" layer="27" rot="R90" display="off"/>
+</element>
 </elements>
 <signals>
@@
 <contactref element="OPTO1" pad="NPN_C"/>
 <contactref element="R2" pad="1"/>
-<contactref element="Q1" pad="1"/>
 <wire x1="27.99" y1="5.99" x2="30.2" y2="6" width="0.5" layer="1"/>
 <wire x1="30.2" y1="6" x2="33.67" y2="6" width="0.5" layer="1"/>
-<wire x1="22.94" y1="8.65" x2="17.25" y2="8.65" width="0.5" layer="1"/>
 <wire x1="17.25" y1="8.65" x2="17.2" y2="8.7" width="0.3" layer="1"/>
-<wire x1="22.94" y1="8.65" x2="23.35" y2="8.65" width="0.3" layer="1"/>
 <wire x1="23.35" y1="8.65" x2="26.01" y2="5.99" width="0.5" layer="1"/>
 <wire x1="27.99" y1="5.99" x2="26.01" y2="5.99" width="0.5" layer="1"/>
@@
 <wire x1="18" y1="6.8" x2="17.2" y2="7.6" width="0.5" layer="1"/>
 <wire x1="17.2" y1="7.6" x2="17.2" y2="8.7" width="0.5" layer="1"/>
+<contactref element="Q2" pad="1"/>
+<wire x1="22.5" y1="8.65" x2="21.45" y2="8.65" width="0.4064" layer="1"/>
+<wire x1="21.45" y1="8.65" x2="20.6" y2="7.8" width="0.4064" layer="1"/>
+<wire x1="20.6" y1="7.8" x2="19.6" y2="7.8" width="0.4064" layer="1"/>
+<wire x1="19.6" y1="7.8" x2="18.7" y2="8.7" width="0.4064" layer="1"/>
+<wire x1="17.2" y1="8.7" x2="18.7" y2="8.7" width="0.4064" layer="1"/>
+<wire x1="22.5" y1="8.65" x2="23.35" y2="8.65" width="0.4064" layer="1"/>
 </signal>
 <signal name="N$4">
@@
 <contactref element="OPTO1" pad="LED_K"/>
 <contactref element="OPTO1" pad="NPN_E"/>
-<contactref element="Q1" pad="2"/>
 <wire x1="27.99" y1="7.99" x2="30.2" y2="8" width="1" layer="1"/>
 <wire x1="30.2" y1="8" x2="33.67" y2="8.54" width="1" layer="1"/>
@@
 <wire x1="26.21" y1="7.99" x2="24.9" y2="9.3" width="0.5" layer="1"/>
 <wire x1="24.9" y1="9.3" x2="23.65" y2="10.55" width="0.5" layer="1"/>
-<wire x1="22.94" y1="10.55" x2="23.65" y2="10.55" width="0.3" layer="1"/>
 <wire x1="16.55" y1="5.27" x2="16.55" y2="6.95" width="0.5" layer="16"/>
 <wire x1="16.55" y1="6.95" x2="19.2" y2="9.6" width="0.5" layer="16"/>
@@
 <wire x1="24.6" y1="9.6" x2="24.9" y2="9.3" width="0.5" layer="16"/>
 <via x="24.9" y="9.3" extent="1-16" drill="0.5"/>
+<contactref element="Q2" pad="2"/>
+<wire x1="22.5" y1="10.55" x2="23.65" y2="10.55" width="0.4064" layer="1"/>
 </signal>
 <signal name="N$2">
-<contactref element="Q1" pad="3"/>
 <contactref element="LED1" pad="C"/>
-<wire x1="20.74" y1="9.6" x2="16.2" y2="9.6" width="0.5" layer="1"/>
 <wire x1="16.2" y1="9.6" x2="15.32" y2="8.72" width="0.5" layer="1"/>
 <wire x1="14.25" y1="8.72" x2="15.32" y2="8.72" width="0.5" layer="1"/>
+<contactref element="Q2" pad="3"/>
+<wire x1="16.2" y1="9.6" x2="20.3" y2="9.6" width="0.4064" layer="1"/>
 </signal>
 <signal name="N$3">

Commit message: Moving STL's over here
Parts:
- removed J2: (no value), !con-lstb:MA03-1
- J1: value CONN-RECT-3PINJST_PH_2MM -> CONN-0.1-S-1X3; device FirePick:CONN-JST_PH-2.0MM-3PIN-SMT-RA -> !con-lstb:MA03-1
- LED1: value (none) -> AMBER
- moved J1 27.7 mm to (2.50, 5.40)
- moved LOGO5 16.1 mm to (29.4, 7.78), flipped to the top
- moved LOGO6 8.17 mm to (7.40, 0.49), flipped to the top, turned to 90 degrees
- moved R3 8.01 mm to (16.6, 9.20)
- moved OPTO1 7.26 mm to (20.0, 3.60)
- moved LED1 7.25 mm to (20.0, 8.62)
- moved FID4 7.18 mm to (28.1, 8.04)
- moved LOGO4 6.20 mm to (30.6, 8.99)
- moved R1 5.22 mm to (11.0, 9.20), turned to 90 degrees
- moved Q2 4.10 mm to (25.4, 8.70), turned to 0 degrees
- moved R2 3.32 mm to (13.9, 9.20)
- moved FID3 1.79 mm to (2.50, 10.0)
Connections:
- net 5V: no longer J2.1
- net GND: no longer J2.3
- net OPTO_OUT: no longer J2.2
Routing:
- net 5V: track 41.7 -> 15.0 mm, vias 1 -> 0
- net OPTO_OUT: track 25.6 -> 39.2 mm
- net N$4: track 10.2 -> 6.62 mm
- net N$2: track 6.41 -> 4.39 mm
- net GND: track 32.2 -> 33.6 mm, vias 1 -> 0
- net N$3: track 2.65 -> 2.03 mm
Other:
- board size 35.3 x 12 mm -> 33 x 11 mm
- board text added: "G"
- board text added: "S"
