File: electronics/eopto01/EAGLE/EOPTO01.sch (EAGLE design)
At the start: 13 parts, among them J1 CONN-RECT-3PINJST_PH_2MM, Q1 BC849

Commit message: Revision A, after assembling first batch of PCBs.
Parts:
- removed Q1: BC849, transistor:BC849
- added Q2: BSS138, SparkFun-DiscreteSemi:MOSFET-NCHANNELBSS138
- R1: value (none) -> 120
- R2: value (none) -> 10k
- R3: value (none) -> 1k
Connections:
- net GND: now also Q2.S; no longer Q1.E
- net N$2: now also Q2.D; no longer Q1.C
- net OPTO_OUT: now also Q2.G; no longer Q1.B
Changed lines of the file:
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@@
 <part name="J1" library="FirePick" deviceset="CONN-RECT-3PIN" device="JST_PH_2MM"/>
 <part name="J2" library="!con-lstb" deviceset="MA03-1" device=""/>
-<part name="R1" library="SparkFun-Resistors" deviceset="RESISTOR" device="0805-RES"/>
-<part name="R2" library="SparkFun-Resistors" deviceset="RESISTOR" device="0805-RES"/>
-<part name="R3" library="SparkFun-Resistors" deviceset="RESISTOR" device="0805-RES"/>
+<part name="R1" library="SparkFun-Resistors" deviceset="RESISTOR" device="0805-RES" value="120"/>
+<part name="R2" library="SparkFun-Resistors" deviceset="RESISTOR" device="0805-RES" value="10k"/>
+<part name="R3" library="SparkFun-Resistors" deviceset="RESISTOR" device="0805-RES" value="1k"/>
 <part name="LED1" library="SparkFun-LED" deviceset="LED" device="1206"/>
-<part name="Q1" library="transistor" deviceset="BC849" device=""/>
 <part name="SUPPLY1" library="SparkFun-Aesthetics" deviceset="5V" device=""/>
 <part name="SUPPLY2" library="SparkFun-Aesthetics" deviceset="5V" device=""/>
@@
 <part name="GND5" library="SparkFun-Aesthetics" deviceset="GND" device=""/>
 <part name="SUPPLY4" library="SparkFun-Aesthetics" deviceset="5V" device=""/>
+<part name="Q2" library="SparkFun-DiscreteSemi" deviceset="MOSFET-NCHANNEL" device="BSS138" value="BSS138"/>
 </parts>
 <sheets>
@@
 <instance part="R3" gate="G$1" x="259.08" y="162.56" rot="R90"/>
 <instance part="LED1" gate="G$1" x="259.08" y="152.4"/>
-<instance part="Q1" gate="G$1" x="256.54" y="137.16"/>
 <instance part="SUPPLY1" gate="G$1" x="198.12" y="172.72"/>
 <instance part="SUPPLY2" gate="G$1" x="259.08" y="172.72"/>
@@
 <instance part="GND5" gate="1" x="109.22" y="119.38"/>
 <instance part="SUPPLY4" gate="G$1" x="109.22" y="172.72"/>
+<instance part="Q2" gate="G$1" x="259.08" y="137.16"/>
 </instances>
 <busses>
@@
 </segment>
 <segment>
-<pinref part="Q1" gate="G$1" pin="B"/>
-<wire x1="254" y1="137.16" x2="233.68" y2="137.16" width="0.1524" layer="91"/>
 <label x="236.22" y="137.16" size="1.778" layer="95"/>
+<pinref part="Q2" gate="G$1" pin="G"/>
+<wire x1="251.46" y1="137.16" x2="233.68" y2="137.16" width="0.1524" layer="91"/>
 </segment>
 </net>
@@
 </segment>
 <segment>
-<pinref part="Q1" gate="G$1" pin="E"/>
 <pinref part="GND3" gate="1" pin="GND"/>
 <wire x1="259.08" y1="132.08" x2="259.08" y2="121.92" width="0.1524" layer="91"/>
+<pinref part="Q2" gate="G$1" pin="S"/>
 </segment>
 </net>
 <net name="N$2" class="0">
 <segment>
-<pinref part="Q1" gate="G$1" pin="C"/>
 <pinref part="LED1" gate="G$1" pin="C"/>
 <wire x1="259.08" y1="142.24" x2="259.08" y2="147.32" width="0.1524" layer="91"/>
+<pinref part="Q2" gate="G$1" pin="D"/>
 </segment>
 </net>

Commit message: Moving STL's over here
Parts:
- removed J2: (no value), !con-lstb:MA03-1
- FID3, FID4, LOGO4, LOGO5, LOGO6: BOM (none) -> EXCLUDE
- J1: value CONN-RECT-3PINJST_PH_2MM -> CONN-0.1-S-1X3; device FirePick:CONN-RECT-3PINJST_PH_2MM -> !con-lstb:MA03-1; PARTNO (none) -> CONN-0.1-RA-1X3
- LED1: value (none) -> AMBER; PARTNO (none) -> LTST-C150AKT
- OPTO1: PARTNO (none) -> TCST2103
- Q2: PARTNO (none) -> BSS138
- R1: PARTNO (none) -> RC0805FR-07120RL
- R2: PARTNO (none) -> RC0805FR-0710KL
- R3: PARTNO (none) -> RC0805FR-071KL
Connections:
- net 5V: no longer J2.1
- net GND: no longer J2.3
- net OPTO_OUT: no longer J2.2
Changed lines of the file:
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@@
 <?xml version="1.0" encoding="utf-8"?>
 <!DOCTYPE eagle SYSTEM "eagle.dtd">
-<eagle version="7.1.0">
+<eagle version="7.2.0">
 <drawing>
 <settings>
@@
 </classes>
 <parts>
-<part name="J1" library="FirePick" deviceset="CONN-RECT-3PIN" device="JST_PH_2MM"/>
-<part name="J2" library="!con-lstb" deviceset="MA03-1" device=""/>
-<part name="R1" library="SparkFun-Resistors" deviceset="RESISTOR" device="0805-RES" value="120"/>
-<part name="R2" library="SparkFun-Resistors" deviceset="RESISTOR" device="0805-RES" value="10k"/>
-<part name="R3" library="SparkFun-Resistors" deviceset="RESISTOR" device="0805-RES" value="1k"/>
-<part name="LED1" library="SparkFun-LED" deviceset="LED" device="1206"/>
+<part name="J1" library="!con-lstb" deviceset="MA03-1" device="" value="CONN-0.1-S-1X3">
+<attribute name="PARTNO" value="CONN-0.1-RA-1X3"/>
+</part>
+<part name="R1" library="SparkFun-Resistors" deviceset="RESISTOR" device="0805-RES" value="120">
+<attribute name="PARTNO" value="RC0805FR-07120RL"/>
+</part>
+<part name="R2" library="SparkFun-Resistors" deviceset="RESISTOR" device="0805-RES" value="10k">
+<attribute name="PARTNO" value="RC0805FR-0710KL"/>
+</part>
+<part name="R3" library="SparkFun-Resistors" deviceset="RESISTOR" device="0805-RES" value="1k">
+<attribute name="PARTNO" value="RC0805FR-071KL"/>
+</part>
+<part name="LED1" library="SparkFun-LED" deviceset="LED" device="1206" value="AMBER">
+<attribute name="PARTNO" value="LTST-C150AKT"/>
+</part>
 <part name="SUPPLY1" library="SparkFun-Aesthetics" deviceset="5V" device=""/>
 <part name="SUPPLY2" library="SparkFun-Aesthetics" deviceset="5V" device=""/>
@@
 <part name="GND3" library="SparkFun-Aesthetics" deviceset="GND" device=""/>
 <part name="GND4" library="SparkFun-Aesthetics" deviceset="GND" device=""/>
-<part name="OPTO1" library="FirePick" deviceset="TCST2103" device=""/>
-<part name="FID3" library="SparkFun-Aesthetics" deviceset="FIDUCIAL" device="1X2"/>
-<part name="FID4" library="SparkFun-Aesthetics" deviceset="FIDUCIAL" device="1X2"/>
+<part name="OPTO1" library="FirePick" deviceset="TCST2103" device="">
+<attribute name="PARTNO" value="TCST2103"/>
+</part>
+<part name="FID3" library="SparkFun-Aesthetics" deviceset="FIDUCIAL" device="1X2">
+<attribute name="BOM" value="EXCLUDE"/>
+</part>
+<part name="FID4" library="SparkFun-Aesthetics" deviceset="FIDUCIAL" device="1X2">
+<attribute name="BOM" value="EXCLUDE"/>
+</part>
 <part name="FRAME1" library="frames" deviceset="A3L-LOC" device=""/>
-<part name="LOGO4" library="FirePick" deviceset="LOGO-FIREPICK" device="MEDIUM" value="LOGO-FIREPICKMEDIUM"/>
-<part name="LOGO5" library="FirePick" deviceset="LOGO-OSHW" device="SMALL" value="LOGO-OSHWSMALL"/>
-<part name="LOGO6" library="FirePick" deviceset="LOGO-CC-BY-SA" device="MEDIUM" value="LOGO-CC-BY-SAMEDIUM"/>
+<part name="LOGO4" library="FirePick" deviceset="LOGO-FIREPICK" device="MEDIUM" value="LOGO-FIREPICKMEDIUM">
+<attribute name="BOM" value="EXCLUDE"/>
+</part>
+<part name="LOGO5" library="FirePick" deviceset="LOGO-OSHW" device="SMALL" value="LOGO-OSHWSMALL">
+<attribute name="BOM" value="EXCLUDE"/>
+</part>
+<part name="LOGO6" library="FirePick" deviceset="LOGO-CC-BY-SA" device="MEDIUM" value="LOGO-CC-BY-SAMEDIUM">
+<attribute name="BOM" value="EXCLUDE"/>
+</part>
 <part name="GND5" library="SparkFun-Aesthetics" deviceset="GND" device=""/>
 <part name="SUPPLY4" library="SparkFun-Aesthetics" deviceset="5V" device=""/>
-<part name="Q2" library="SparkFun-DiscreteSemi" deviceset="MOSFET-NCHANNEL" device="BSS138" value="BSS138"/>
+<part name="Q2" library="SparkFun-DiscreteSemi" deviceset="MOSFET-NCHANNEL" device="BSS138" value="BSS138">
+<attribute name="PARTNO" value="BSS138"/>
+</part>
 </parts>
 <sheets>
@@
 </plain>
 <instances>
-<instance part="J1" gate="G$1" x="83.82" y="134.62" smashed="yes">
-<attribute name="NAME" x="77.47" y="140.462" size="1.778" layer="95"/>
-</instance>
-<instance part="J2" gate="G$1" x="93.98" y="134.62" smashed="yes" rot="MR180">
+<instance part="J1" gate="G$1" x="93.98" y="134.62" smashed="yes" rot="MR180">
 <attribute name="VALUE" x="92.71" y="142.24" size="1.778" layer="96" rot="MR180"/>
-</instance>
-<instance part="R1" gate="G$1" x="142.24" y="162.56" rot="R90"/>
-<instance part="R2" gate="G$1" x="198.12" y="162.56" rot="R90"/>
-<instance part="R3" gate="G$1" x="259.08" y="162.56" rot="R90"/>
-<instance part="LED1" gate="G$1" x="259.08" y="152.4"/>
+<attribute name="PARTNO" x="93.98" y="134.62" size="1.778" layer="96" display="off"/>
+</instance>
+<instance part="R1" gate="G$1" x="142.24" y="162.56" rot="R90">
+<attribute name="PARTNO" x="142.24" y="162.56" size="1.778" layer="96" display="off"/>
+</instance>
+<instance part="R2" gate="G$1" x="198.12" y="162.56" rot="R90">
+<attribute name="PARTNO" x="198.12" y="162.56" size="1.778" layer="96" display="off"/>
+</instance>
+<instance part="R3" gate="G$1" x="259.08" y="162.56" rot="R90">
+<attribute name="PARTNO" x="259.08" y="162.56" size="1.778" layer="96" display="off"/>
+</instance>
+<instance part="LED1" gate="G$1" x="259.08" y="152.4">
+<attribute name="PARTNO" x="259.08" y="152.4" size="1.778" layer="96" display="off"/>
+</instance>
 <instance part="SUPPLY1" gate="G$1" x="198.12" y="172.72"/>
 <instance part="SUPPLY2" gate="G$1" x="259.08" y="172.72"/>
@@
 <instance part="GND3" gate="1" x="259.08" y="119.38"/>
 <instance part="GND4" gate="1" x="96.52" y="12.7"/>
-<instance part="OPTO1" gate="G$1" x="167.64" y="134.62"/>
-<instance part="FID3" gate="G$1" x="284.48" y="12.7"/>
-<instance part="FID4" gate="G$1" x="284.48" y="7.62"/>
+<instance part="OPTO1" gate="G$1" x="167.64" y="134.62">
+<attribute name="PARTNO" x="167.64" y="134.62" size="1.778" layer="96" display="off"/>
+</instance>
+<instance part="FID3" gate="G$1" x="284.48" y="12.7">
+<attribute name="BOM" x="284.48" y="12.7" size="1.778" layer="96" display="off"/>
+</instance>
+<instance part="FID4" gate="G$1" x="284.48" y="7.62">
+<attribute name="BOM" x="284.48" y="7.62" size="1.778" layer="96" display="off"/>
+</instance>
 <instance part="FRAME1" gate="G$1" x="0.000003125" y="0"/>
-<instance part="LOGO4" gate="G$1" x="85.09" y="8.89"/>
-<instance part="LOGO5" gate="G$1" x="360.68" y="26.67"/>
-<instance part="LOGO6" gate="G$1" x="3.81" y="3.81"/>
+<instance part="LOGO4" gate="G$1" x="85.09" y="8.89">
+<attribute name="BOM" x="85.09" y="8.89" size="1.778" layer="96" display="off"/>
+</instance>
+<instance part="LOGO5" gate="G$1" x="360.68" y="26.67">
+<attribute name="BOM" x="360.68" y="26.67" size="1.778" layer="96" display="off"/>
+</instance>
+<instance part="LOGO6" gate="G$1" x="3.81" y="3.81">
+<attribute name="BOM" x="3.81" y="3.81" size="1.778" layer="96" display="off"/>
+</instance>
 <instance part="GND5" gate="1" x="109.22" y="119.38"/>
 <instance part="SUPPLY4" gate="G$1" x="109.22" y="172.72"/>
-<instance part="Q2" gate="G$1" x="259.08" y="137.16"/>
+<instance part="Q2" gate="G$1" x="259.08" y="137.16">
+<attribute name="PARTNO" x="259.08" y="137.16" size="1.778" layer="96" display="off"/>
+</instance>
 </instances>
 <busses>
@@
 <segment>
 <pinref part="J1" gate="G$1" pin="2"/>
-<pinref part="J2" gate="G$1" pin="2"/>
-<wire x1="86.36" y1="134.62" x2="101.6" y2="134.62" width="0.1524" layer="91"/>
 <wire x1="101.6" y1="134.62" x2="119.38" y2="134.62" width="0.1524" layer="91"/>
 <label x="111.76" y="134.62" size="1.778" layer="95"/>
@@
 <segment>
 <pinref part="J1" gate="G$1" pin="1"/>
-<pinref part="J2" gate="G$1" pin="1"/>
-<wire x1="86.36" y1="137.16" x2="101.6" y2="137.16" width="0.1524" layer="91"/>
 <wire x1="101.6" y1="137.16" x2="109.22" y2="137.16" width="0.1524" layer="91"/>
 <pinref part="SUPPLY4" gate="G$1" pin="5V"/>
@@
 <segment>
 <pinref part="J1" gate="G$1" pin="3"/>
-<pinref part="J2" gate="G$1" pin="3"/>
-<wire x1="86.36" y1="132.08" x2="101.6" y2="132.08" width="0.1524" layer="91"/>
 <wire x1="101.6" y1="132.08" x2="109.22" y2="132.08" width="0.1524" layer="91"/>
 <pinref part="GND5" gate="1" pin="GND"/>
